File: schema_keyboard_game.kicad_sch (KiCad schematic)
At the start: 6 parts, among them SW1 SW_Push, SW2 SW_Push, SW3 SW_Push, SW4 SW_Push, U1 ESP32-S3-DevKitC

Commit message: ver 1
Parts:
- added C1, C10, C100, C11, C12, C13, C14, C15, C16, C17, C18, C19, C2, C20, C21, C22, C23, C24, C25, C26, C27, C28, C29, C3, C30, C31, C32, C33, C34, C35, C36, C37, C38, C39, C4, C40, C41, C42, C43, C44, C45, C46, C47, C48, C49, C5, C50, C51, C52, C53, C54, C55, C56, C57, C58, C59, C6, C60, C61, C62, C63, C64, C65, C66, C67, C68, C69, C7, C70, C71, C72, C73, C74, C75, C76, C77, C78, C79, C8, C80, C81, C82, C83, C84, C85, C86, C87, C88, C89, C9, C90, C91, C92, C93, C94, C95, C96, C97, C98, C99: C, symbol Device:C
- added D1, D10, D100, D11, D12, D13, D14, D15, D16, D17, D18, D19, D2, D20, D21, D22, D23, D24, D25, D26, D27, D28, D29, D3, D30, D31, D32, D33, D34, D35, D36, D37, D38, D39, D4, D40, D41, D42, D43, D44, D45, D46, D47, D48, D49, D5, D50, D51, D52, D53, D54, D55, D56, D57, D58, D59, D6, D60, D61, D62, D63, D64, D65, D66, D67, D68, D69, D7, D70, D71, D72, D73, D74, D75, D76, D77, D78, D79, D8, D80, D81, D82, D83, D84, D85, D86, D87, D88, D89, D9, D90, D91, D92, D93, D94, D95, D96, D97, D98, D99: WS2812B, LED_SMD:LED_WS2812B_PLCC4_5.0x5.0mm_P3.2mm, symbol LED:WS2812B
- added SW10, SW100, SW12, SW13, SW14, SW15, SW16, SW17, SW18, SW19, SW2, SW20, SW22, SW23, SW24, SW25, SW26, SW27, SW28, SW29, SW3, SW30, SW32, SW33, SW34, SW35, SW36, SW37, SW38, SW39, SW4, SW40, SW41, SW42, SW43, SW44, SW45, SW46, SW47, SW48, SW49, SW5, SW50, SW51, SW52, SW53, SW54, SW55, SW56, SW57, SW58, SW59, SW6, SW60, SW61, SW62, SW63, SW64, SW65, SW66, SW67, SW68, SW69, SW7, SW70, SW71, SW72, SW73, SW74, SW75, SW76, SW77, SW78, SW79, SW8, SW80, SW81, SW82, SW83, SW84, SW85, SW86, SW87, SW88, SW89, SW9, SW90, SW91, SW92, SW93, SW94, SW95, SW96, SW97, SW98, SW99: SW_Push, Button_Switch_Keyboard:SW_Cherry_MX_1.00u_Plate, symbol Switch:SW_Push
- LCD1: Spice_Netlist_Enabled Y -> (none)
- renumbered SW2 to SW11, SW3 to SW21, SW4 to SW31
Connections:
- net row_1: now reaches SW11.1
- net row_1: now also SW1.1, SW21.1, SW31.1, U1.41 (GPIO1/ADC1_CH0), SW41.1, SW51.1, SW61.1, SW71.1, SW81.1, SW91.1
- net cl_2: now reaches SW11.2
- net cl_2: now also U1.20 (GPIO14/ADC2_CH3), SW12.2, SW13.2, SW14.2, SW15.2, SW16.2, SW17.2, SW18.2, SW19.2, SW20.2
- net cl_4: now reaches SW31.2
- net cl_4: now also U1.11 (GPIO18/ADC2_CH7), SW32.2, SW33.2, SW34.2, SW35.2, SW36.2, SW37.2, SW38.2, SW39.2, SW40.2
- net cl_1: now reaches SW1.2
- net cl_1: now also U1.19 (GPIO13/ADC2_CH2), SW10.2, SW2.2, SW3.2, SW4.2, SW5.2, SW6.2, SW7.2, SW8.2, SW9.2
- net +3V3: now reaches U1.1 (3V3), U1.2 (3V3)
- net +3V3: now also LCD1.1 (GND)
- net cl_3: now reaches U1.10 (GPIO17/ADC2_CH6)
- net cl_3: now also SW21.2, SW22.2, SW23.2, SW24.2, SW25.2, SW26.2, SW27.2, SW28.2, SW29.2, SW30.2
- net row_6: now reaches U1.12 (GPIO8/ADC1_CH7)
- net row_6: now also SW16.1, SW26.1, SW36.1, SW46.1, SW56.1, SW6.1, SW66.1, SW76.1, SW86.1, SW96.1
- net row_3: now reaches U1.13 (GPIO3/ADC1_CH2)
- net row_3: now also SW13.1, SW23.1, SW3.1, SW33.1, SW43.1, SW53.1, SW63.1, SW73.1, SW83.1, SW93.1
- net cl_10: now reaches U1.14 (GPIO46)
- net cl_10: now also SW100.2, SW91.2, SW92.2, SW93.2, SW94.2, SW95.2, SW96.2, SW97.2, SW98.2, SW99.2
- net row_7: now reaches U1.15 (GPIO9/ADC1_CH8)
- net row_7: now also SW17.1, SW27.1, SW37.1, SW47.1, SW57.1, SW67.1, SW7.1, SW77.1, SW87.1, SW97.1
- net row_8: now reaches U1.16 (GPIO10/ADC1_CH9)
- net row_8: now also SW18.1, SW28.1, SW38.1, SW48.1, SW58.1, SW68.1, SW78.1, SW8.1, SW88.1, SW98.1
- net row_9: now reaches U1.17 (GPIO11/ADC2_CH0)
- net row_9: now also SW19.1, SW29.1, SW39.1, SW49.1, SW59.1, SW69.1, SW79.1, SW89.1, SW9.1, SW99.1
- net row_10: now reaches U1.18 (GPIO12/ADC2_CH1)
- net row_10: now also SW10.1, SW100.1, SW20.1, SW30.1, SW40.1, SW50.1, SW60.1, SW70.1, SW80.1, SW90.1
- net +5V: now reaches U1.21 (5V)
- net +5V: now also C1.1, C10.1, C100.1, C11.1, C12.1, C13.1, C14.1, C15.1, C16.1, C17.1, C18.1, C19.1, C2.1, C20.1, C21.1, C22.1, C23.1, C24.1, C25.1, C26.1, C27.1, C28.1, C29.1, C3.1, C30.1, C31.1, C32.1, C33.1, C34.1, C35.1, C36.1, C37.1, C38.1, C39.1, C4.1, C40.1, C41.1, C42.1, C43.1, C44.1, C45.1, C46.1, C47.1, C48.1, C49.1, C5.1, C50.1, C51.1, C52.1, C53.1, C54.1, C55.1, C56.1, C57.1, C58.1, C59.1, C6.1, C60.1, C61.1, C62.1, C63.1, C64.1, C65.1, C66.1, C67.1, C68.1, C69.1, C7.1, C70.1, C71.1, C72.1, C73.1, C74.1, C75.1, C76.1, C77.1, C78.1, C79.1, C8.1, C80.1, C81.1, C82.1, C83.1, C84.1, C85.1, C86.1, C87.1, C88.1, C89.1, C9.1, C90.1, C91.1, C92.1, C93.1, C94.1, C95.1, C96.1, C97.1, C98.1, C99.1, D1.1 (VDD), D10.1 (VDD), D100.1 (VDD), D11.1 (VDD), D12.1 (VDD), D13.1 (VDD), D14.1 (VDD), D15.1 (VDD), D16.1 (VDD), D17.1 (VDD), D18.1 (VDD), D19.1 (VDD), D2.1 (VDD), D20.1 (VDD), D21.1 (VDD), D22.1 (VDD), D23.1 (VDD), D24.1 (VDD), D25.1 (VDD), D26.1 (VDD), D27.1 (VDD), D28.1 (VDD), D29.1 (VDD), D3.1 (VDD), D30.1 (VDD), D31.1 (VDD), D32.1 (VDD), D33.1 (VDD), D34.1 (VDD), D35.1 (VDD), D36.1 (VDD), D37.1 (VDD), D38.1 (VDD), D39.1 (VDD), D4.1 (VDD), D40.1 (VDD), D41.1 (VDD), D42.1 (VDD), D43.1 (VDD), D44.1 (VDD), D45.1 (VDD), D46.1 (VDD), D47.1 (VDD), D48.1 (VDD), D49.1 (VDD), D5.1 (VDD), D50.1 (VDD), D51.1 (VDD), D52.1 (VDD), D53.1 (VDD), D54.1 (VDD), D55.1 (VDD), D56.1 (VDD), D57.1 (VDD), D58.1 (VDD), D59.1 (VDD), D6.1 (VDD), D60.1 (VDD), D61.1 (VDD), D62.1 (VDD), D63.1 (VDD), D64.1 (VDD), D65.1 (VDD), D66.1 (VDD), D67.1 (VDD), D68.1 (VDD), D69.1 (VDD), D7.1 (VDD), D70.1 (VDD), D71.1 (VDD), D72.1 (VDD), D73.1 (VDD), D74.1 (VDD), D75.1 (VDD), D76.1 (VDD), D77.1 (VDD), D78.1 (VDD), D79.1 (VDD), D8.1 (VDD), D80.1 (VDD), D81.1 (VDD), D82.1 (VDD), D83.1 (VDD), D84.1 (VDD), D85.1 (VDD), D86.1 (VDD), D87.1 (VDD), D88.1 (VDD), D89.1 (VDD), D9.1 (VDD), D90.1 (VDD), D91.1 (VDD), D92.1 (VDD), D93.1 (VDD), D94.1 (VDD), D95.1 (VDD), D96.1 (VDD), D97.1 (VDD), D98.1 (VDD), D99.1 (VDD)
- net GND: now reaches U1.22 (GND), U1.23 (GND), U1.24 (GND), U1.44 (GND)
- net GND: now also LCD1.1 (GND), C1.2, C10.2, C100.2, C11.2, C12.2, C13.2, C14.2, C15.2, C16.2, C17.2, C18.2, C19.2, C2.2, C20.2, C21.2, C22.2, C23.2, C24.2, C25.2, C26.2, C27.2, C28.2, C29.2, C3.2, C30.2, C31.2, C32.2, C33.2, C34.2, C35.2, C36.2, C37.2, C38.2, C39.2, C4.2, C40.2, C41.2, C42.2, C43.2, C44.2, C45.2, C46.2, C47.2, C48.2, C49.2, C5.2, C50.2, C51.2, C52.2, C53.2, C54.2, C55.2, C56.2, C57.2, C58.2, C59.2, C6.2, C60.2, C61.2, C62.2, C63.2, C64.2, C65.2, C66.2, C67.2, C68.2, C69.2, C7.2, C70.2, C71.2, C72.2, C73.2, C74.2, C75.2, C76.2, C77.2, C78.2, C79.2, C8.2, C80.2, C81.2, C82.2, C83.2, C84.2, C85.2, C86.2, C87.2, C88.2, C89.2, C9.2, C90.2, C91.2, C92.2, C93.2, C94.2, C95.2, C96.2, C97.2, C98.2, C99.2, D1.3 (VSS), D10.3 (VSS), D100.3 (VSS), D11.3 (VSS), D12.3 (VSS), D13.3 (VSS), D14.3 (VSS), D15.3 (VSS), D16.3 (VSS), D17.3 (VSS), D18.3 (VSS), D19.3 (VSS), D2.3 (VSS), D20.3 (VSS), D21.3 (VSS), D22.3 (VSS), D23.3 (VSS), D24.3 (VSS), D25.3 (VSS), D26.3 (VSS), D27.3 (VSS), D28.3 (VSS), D29.3 (VSS), D3.3 (VSS), D30.3 (VSS), D31.3 (VSS), D32.3 (VSS), D33.3 (VSS), D34.3 (VSS), D35.3 (VSS), D36.3 (VSS), D37.3 (VSS), D38.3 (VSS), D39.3 (VSS), D4.3 (VSS), D40.3 (VSS), D41.3 (VSS), D42.3 (VSS), D43.3 (VSS), D44.3 (VSS), D45.3 (VSS), D46.3 (VSS), D47.3 (VSS), D48.3 (VSS), D49.3 (VSS), D5.3 (VSS), D50.3 (VSS), D51.3 (VSS), D52.3 (VSS), D53.3 (VSS), D54.3 (VSS), D55.3 (VSS), D56.3 (VSS), D57.3 (VSS), D58.3 (VSS), D59.3 (VSS), D6.3 (VSS), D60.3 (VSS), D61.3 (VSS), D62.3 (VSS), D63.3 (VSS), D64.3 (VSS), D65.3 (VSS), D66.3 (VSS), D67.3 (VSS), D68.3 (VSS), D69.3 (VSS), D7.3 (VSS), D70.3 (VSS), D71.3 (VSS), D72.3 (VSS), D73.3 (VSS), D74.3 (VSS), D75.3 (VSS), D76.3 (VSS), D77.3 (VSS), D78.3 (VSS), D79.3 (VSS), D8.3 (VSS), D80.3 (VSS), D81.3 (VSS), D82.3 (VSS), D83.3 (VSS), D84.3 (VSS), D85.3 (VSS), D86.3 (VSS), D87.3 (VSS), D88.3 (VSS), D89.3 (VSS), D9.3 (VSS), D90.3 (VSS), D91.3 (VSS), D92.3 (VSS), D93.3 (VSS), D94.3 (VSS), D95.3 (VSS), D96.3 (VSS), D97.3 (VSS), D98.3 (VSS), D99.3 (VSS)
- net cl_5: now reaches U1.27 (GPIO21)
- net cl_5: now also SW41.2, SW42.2, SW43.2, SW44.2, SW45.2, SW46.2, SW47.2, SW48.2, SW49.2, SW50.2
- net cl_9: now reaches U1.35 (GPIO38)
- net cl_9: now also SW81.2, SW82.2, SW83.2, SW84.2, SW85.2, SW86.2, SW87.2, SW88.2, SW89.2, SW90.2
- net dc: now reaches U1.36 (GPIO39/MTCK)
- net dc: now also LCD1.6 (DC)
- net reset_tft: now reaches U1.37 (GPIO40/MTDO)
- net reset_tft: now also LCD1.5 (RES)
- net backlight: now reaches U1.38 (GPIO41/MTDI)
- net backlight: now also LCD1.7 (BLK)
- net cl_8: now reaches U1.39 (GPIO42/MTMS)
- net cl_8: now also SW71.2, SW72.2, SW73.2, SW74.2, SW75.2, SW76.2, SW77.2, SW78.2, SW79.2, SW80.2
- net row_4: now reaches U1.4 (GPIO4/ADC1_CH3)
- net row_4: now also SW14.1, SW24.1, SW34.1, SW4.1, SW44.1, SW54.1, SW64.1, SW74.1, SW84.1, SW94.1
- net row_2: now reaches U1.40 (GPIO2/ADC1_CH1)
- net row_2: now also SW12.1, SW2.1, SW22.1, SW32.1, SW42.1, SW52.1, SW62.1, SW72.1, SW82.1, SW92.1
- net row_5: now reaches U1.5 (GPIO5/ADC1_CH4)
- net row_5: now also SW15.1, SW25.1, SW35.1, SW45.1, SW5.1, SW55.1, SW65.1, SW75.1, SW85.1, SW95.1
- net sda: now reaches U1.6 (GPIO6/ADC1_CH5)
- net sda: now also LCD1.4 (SDA)
- net sck: now reaches U1.7 (GPIO7/ADC1_CH6)
- net sck: now also LCD1.3 (SCK)
- net cl_6: now reaches U1.8 (GPIO15/ADC2_CH4/32K_P)
- net cl_6: now also SW51.2, SW52.2, SW53.2, SW54.2, SW55.2, SW56.2, SW57.2, SW58.2, SW59.2, SW60.2
- net cl_7: now reaches U1.9 (GPIO16/ADC2_CH5/32K_N)
- net cl_7: now also SW61.2, SW62.2, SW63.2, SW64.2, SW65.2, SW66.2, SW67.2, SW68.2, SW69.2, SW70.2
- new net: D16.2 (DOUT), D26.4 (DIN)
- new net: D16.4 (DIN), D6.2 (DOUT)
- new net: D82.2 (DOUT), D92.4 (DIN)
- new net: D72.2 (DOUT), D82.4 (DIN)
- new net: D1.2 (DOUT), D11.4 (DIN)
- new net: D100.4 (DIN), D90.2 (DOUT)
- new net: D26.2 (DOUT), D36.4 (DIN)
- new net: D24.2 (DOUT), D34.4 (DIN)
- new net: D14.2 (DOUT), D24.4 (DIN)
- new net: D17.4 (DIN), D7.2 (DOUT)
- new net: D34.2 (DOUT), D44.4 (DIN)
- new net: D49.2 (DOUT), D59.4 (DIN)
- new net: D39.2 (DOUT), D49.4 (DIN)
- new net: D37.2 (DOUT), D47.4 (DIN)
- new net: D27.2 (DOUT), D37.4 (DIN)
- new net: D14.4 (DIN), D4.2 (DOUT)
- new net: D19.4 (DIN), D9.2 (DOUT)
- new net: D53.2 (DOUT), D63.4 (DIN)
- new net: D43.2 (DOUT), D53.4 (DIN)
- new net: D89.2 (DOUT), D99.4 (DIN)
- new net: D42.2 (DOUT), D52.4 (DIN)
- new net: D32.2 (DOUT), D42.4 (DIN)
- new net: D84.2 (DOUT), D94.4 (DIN)
- new net: D87.2 (DOUT), D97.4 (DIN)
- new net: D77.2 (DOUT), D87.4 (DIN)
- new net: D30.2 (DOUT), D40.4 (DIN)
- new net: D20.2 (DOUT), D30.4 (DIN)
- new net: D52.2 (DOUT), D62.4 (DIN)
- new net: D78.2 (DOUT), D88.4 (DIN)
- new net: D68.2 (DOUT), D78.4 (DIN)
- new net: D80.2 (DOUT), D90.4 (DIN)
- new net: D70.2 (DOUT), D80.4 (DIN)
- new net: D21.2 (DOUT), D31.4 (DIN)
- new net: D11.2 (DOUT), D21.4 (DIN)
- new net: D18.4 (DIN), D8.2 (DOUT)
- new net: D15.4 (DIN), D5.2 (DOUT)
- new net: D69.2 (DOUT), D79.4 (DIN)
- new net: D59.2 (DOUT), D69.4 (DIN)
- new net: D22.2 (DOUT), D32.4 (DIN)
- new net: D12.2 (DOUT), D22.4 (DIN)
- new net: D33.2 (DOUT), D43.4 (DIN)
- new net: D56.2 (DOUT), D66.4 (DIN)
- new net: D46.2 (DOUT), D56.4 (DIN)
- new net: D23.2 (DOUT), D33.4 (DIN)
- new net: D13.2 (DOUT), D23.4 (DIN)
- new net: D19.2 (DOUT), D29.4 (DIN)
- new net: D54.2 (DOUT), D64.4 (DIN)
- new net: D44.2 (DOUT), D54.4 (DIN)
- new net: D28.2 (DOUT), D38.4 (DIN)
- new net: D18.2 (DOUT), D28.4 (DIN)
- new net: D12.4 (DIN), D2.2 (DOUT)
- new net: D36.2 (DOUT), D46.4 (DIN)
- new net: D76.2 (DOUT), D86.4 (DIN)
- new net: D66.2 (DOUT), D76.4 (DIN)
- new net: D83.2 (DOUT), D93.4 (DIN)
- new net: D85.2 (DOUT), D95.4 (DIN)
- new net: D75.2 (DOUT), D85.4 (DIN)
- new net: D31.2 (DOUT), D41.4 (DIN)
- new net: D10.2 (DOUT), D20.4 (DIN)
- new net: D62.2 (DOUT), D72.4 (DIN)
- new net: D79.2 (DOUT), D89.4 (DIN)
- new net: D86.2 (DOUT), D96.4 (DIN)
- new net: D67.2 (DOUT), D77.4 (DIN)
- new net: D65.2 (DOUT), D75.4 (DIN)
- new net: D57.2 (DOUT), D67.4 (DIN)
- new net: D47.2 (DOUT), D57.4 (DIN)
- new net: D13.4 (DIN), D3.2 (DOUT)
- new net: D73.2 (DOUT), D83.4 (DIN)
- new net: D63.2 (DOUT), D73.4 (DIN)
- new net: D74.2 (DOUT), D84.4 (DIN)
- new net: D64.2 (DOUT), D74.4 (DIN)
- new net: D88.2 (DOUT), D98.4 (DIN)
- new net: D50.2 (DOUT), D60.4 (DIN)
- new net: D40.2 (DOUT), D50.4 (DIN)
- new net: D60.2 (DOUT), D70.4 (DIN)
- new net: D58.2 (DOUT), D68.4 (DIN)
- new net: D81.2 (DOUT), D91.4 (DIN)
- new net: D48.2 (DOUT), D58.4 (DIN)
- new net: D38.2 (DOUT), D48.4 (DIN)
- new net: D55.2 (DOUT), D65.4 (DIN)
- new net: D45.2 (DOUT), D55.4 (DIN)
- new net: D17.2 (DOUT), D27.4 (DIN)
- new net: D35.2 (DOUT), D45.4 (DIN)
- new net: D25.2 (DOUT), D35.4 (DIN)
- new net: D41.2 (DOUT), D51.4 (DIN)
- new net: D29.2 (DOUT), D39.4 (DIN)
- new net: D61.2 (DOUT), D71.4 (DIN)
- new net: D51.2 (DOUT), D61.4 (DIN)
- new net: D71.2 (DOUT), D81.4 (DIN)
- new net: D15.2 (DOUT), D25.4 (DIN)
- new net led_1: D2.4 (DIN), D91.2 (DOUT)
- new net led_2: D3.4 (DIN), D92.2 (DOUT)
- new net led_3: D4.4 (DIN), D93.2 (DOUT)
- new net led_4: D5.4 (DIN), D94.2 (DOUT)
- new net led_5: D6.4 (DIN), D95.2 (DOUT)
- new net led_6: D7.4 (DIN), D96.2 (DOUT)
- new net led_7: D8.4 (DIN), D97.2 (DOUT)
- new net led_8: D9.4 (DIN), D98.2 (DOUT)
- new net led_9: D10.4 (DIN), D99.2 (DOUT)
- new net rgb_in: D1.4 (DIN)
- new net rgb_out: D100.2 (DOUT)
- no-connect marks 0 -> 12
Other:
- moved on the sheet: SW1, SW11, SW21, SW31, U1

Commit message: ver 1.1 shema
Parts:
- added R1: 470 OM, symbol Device:R
Connections:
- net backlight: no longer U1.38 (GPIO41/MTDI)
- net rgb_in: now also R1.1
- net rgb_out: no longer names the net of D100.2 (DOUT)
- new net: R1.2, U1.38 (GPIO41/MTDI)
- no-connect marks 12 -> 13
Changed lines of the file:
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@@
 	)
 	(no_connect
+		(at 542.29 356.87)
+	)
+	(no_connect
 		(at 140.97 321.31)
 	)
@@
 	(wire
 		(pts
+			(xy 81.28 270.51) (xy 90.17 270.51)
+		)
+		(stroke
+			(width 0)
+			(type default)
+		)
+	)
+	(wire
+		(pts
 			(xy 266.7 62.23) (xy 271.78 62.23)
 		)
@@
 	(wire
 		(pts
+			(xy 69.85 270.51) (xy 73.66 270.51)
+		)
+		(stroke
+			(width 0)
+			(type default)
+		)
+	)
+	(wire
+		(pts
 			(xy 425.45 215.9) (xy 439.42 215.9)
 		)
@@
 		)
 	)
-	(label "rgb_out"
-		(at 542.29 356.87 0)
-		(effects
-			(font
-				(size 1.27 1.27)
-			)
-			(justify left bottom)
-		)
-	)
 	(label "cl_8"
 		(at 165.1 110.49 90)
@@
 		)
 	)
-	(label "backlight"
-		(at 90.17 270.51 180)
+	(label "rgb_in"
+		(at 69.85 270.51 180)
 		(effects
 			(font
@@
 					(unit 1)
 				)
+			)
+		)
+	)
+	(symbol
+		(lib_id "Device:R")
+		(at 77.47 270.51 90)
+		(unit 1)
+		(exclude_from_sim no)
+		(in_bom yes)
+		(on_board yes)
+		(dnp no)
+		(fields_autoplaced yes)
+		(property "Reference" "R1"
+			(at 77.47 264.16 90)
+			(effects
+				(font
+					(size 1.27 1.27)
+				)
+			)
+		)
+		(property "Value" "470 OM"
+			(at 77.47 266.7 90)
+			(effects
+				(font
+					(size 1.27 1.27)
+				)
+			)
+		)
+		(property "Footprint" ""
+			(at 77.47 272.288 90)
+			(effects
+				(font
+					(size 1.27 1.27)
+				)
+				(hide yes)
+			)
+		)
+		(property "Datasheet" "~"
+			(at 77.47 270.51 0)
+			(effects
+				(font
+					(size 1.27 1.27)
+				)
+				(hide yes)
+			)
+		)
+		(property "Description" "Resistor"
+			(at 77.47 270.51 0)
+			(effects
+				(font
+					(size 1.27 1.27)
+				)
+				(hide yes)
+			)
+		)
+		(pin "1"
+		)
+		(pin "2"
+		)
+		(instances
+			(project "schema_keyboard_game"
+				(path "/a48886e6-db89-45aa-9ff6-6672930f6948"
+					(reference "R1")
+					(unit 1)
+				)

Commit message: ver 1.2 schema
Parts:
- added D101, D102, D103, D104, D105, D106, D107, D108, D109, D110: D, symbol Device:D
- added R10, R11, R12, R2, R3, R4, R5, R6, R7, R8, R9: 4.7 kOM, symbol Device:R
Connections:
- net +3V3: now also R12.1
- net cl_1: now also D101.2 (A); no longer U1.19 (GPIO13/ADC2_CH2)
- net cl_10: now also D107.2 (A); no longer U1.14 (GPIO46)
- net cl_2: now also D102.2 (A); no longer U1.20 (GPIO14/ADC2_CH3)
- net cl_3: now also D103.2 (A); no longer U1.10 (GPIO17/ADC2_CH6)
- net cl_4: now also D104.2 (A); no longer U1.11 (GPIO18/ADC2_CH7)
- net cl_5: now also D105.2 (A); no longer U1.27 (GPIO21)
- net cl_6: now also D109.2 (A); no longer U1.8 (GPIO15/ADC2_CH4/32K_P)
- net cl_7: now also D108.2 (A); no longer U1.9 (GPIO16/ADC2_CH5/32K_N)
- net cl_8: now also D110.2 (A); no longer U1.39 (GPIO42/MTMS)
- net cl_9: now also D106.2 (A); no longer U1.35 (GPIO38)
- net row_1: now also R2.2; no longer U1.41 (GPIO1/ADC1_CH0)
- net row_10: now also R11.2; no longer U1.18 (GPIO12/ADC2_CH1)
- net row_2: now also R3.2; no longer U1.40 (GPIO2/ADC1_CH1)
- net row_3: now also R4.2; no longer U1.13 (GPIO3/ADC1_CH2)
- net row_4: now also R5.2; no longer U1.4 (GPIO4/ADC1_CH3)
- net row_5: now also R6.2; no longer U1.5 (GPIO5/ADC1_CH4)
- net row_6: now also R7.2; no longer U1.12 (GPIO8/ADC1_CH7)
- net row_7: now also R8.2; no longer U1.15 (GPIO9/ADC1_CH8)
- net row_8: now also R9.2; no longer U1.16 (GPIO10/ADC1_CH9)
- net row_9: now also R10.2; no longer U1.17 (GPIO11/ADC2_CH0)
- net backlight: no longer names the net of LCD1.7 (BLK)
- net backlight: now also R12.2
- new net: R2.1, U1.41 (GPIO1/ADC1_CH0)
- new net: R9.1, U1.16 (GPIO10/ADC1_CH9)
- new net: D108.1 (K), U1.9 (GPIO16/ADC2_CH5/32K_N)
- new net: D101.1 (K), U1.19 (GPIO13/ADC2_CH2)
- new net: D105.1 (K), U1.27 (GPIO21)
- new net: D102.1 (K), U1.20 (GPIO14/ADC2_CH3)
- new net: R11.1, U1.18 (GPIO12/ADC2_CH1)
- new net: R4.1, U1.13 (GPIO3/ADC1_CH2)
- new net: D109.1 (K), U1.8 (GPIO15/ADC2_CH4/32K_P)
- new net: D107.1 (K), U1.14 (GPIO46)
- new net: D103.1 (K), U1.10 (GPIO17/ADC2_CH6)
- new net: D106.1 (K), U1.35 (GPIO38)
- new net: D104.1 (K), U1.11 (GPIO18/ADC2_CH7)
- new net: R3.1, U1.40 (GPIO2/ADC1_CH1)
- new net: R7.1, U1.12 (GPIO8/ADC1_CH7)
- new net: R6.1, U1.5 (GPIO5/ADC1_CH4)
- new net: D110.1 (K), U1.39 (GPIO42/MTMS)
- new net: R8.1, U1.15 (GPIO9/ADC1_CH8)
- new net: R10.1, U1.17 (GPIO11/ADC2_CH0)
- new net: R5.1, U1.4 (GPIO4/ADC1_CH3)

Commit message: ver 1.3 schema
Parts:
- added C101: 100 nF, Capacitor_SMD:C_1206_3216Metric, symbol Device:C
- added J1: USB_C_Receptacle_PowerOnly_6P, Connector_USB:USB_C_Receptacle_HRO_TYPE-C-31-M-17, symbol Connector:USB_C_Receptacle_PowerOnly_6P
- added R13: 470, Resistor_SMD:R_1206_3216Metric, symbol Device:R
- added SW101: SW_Push, Button_Switch_THT:SW_PUSH_6mm, symbol Switch:SW_Push
- C1: value C -> 100 n; footprint (none) -> Capacitor_SMD:C_1206_3216Metric
- C10, C100, C11, C12, C13, C14, C15, C16, C17, C18, C19, C2, C20, C21, C22, C23, C24, C25, C26, C27, C28, C29, C3, C30, C31, C32, C33, C34, C35, C36, C37, C38, C39, C4, C40, C41, C42, C43, C44, C45, C46, C47, C48, C49, C5, C50, C51, C52, C53, C54, C55, C56, C57, C58, C59, C6, C60, C61, C62, C63, C64, C65, C66, C67, C68, C69, C7, C70, C71, C72, C73, C74, C75, C76, C77, C78, C79, C8, C80, C81, C82, C83, C84, C85, C86, C87, C88, C89, C9, C90, C91, C92, C93, C94, C95, C96, C97, C98, C99: footprint (none) -> Capacitor_SMD:C_1206_3216Metric
- D101, D102, D103, D104, D105, D106, D107, D108, D109, D110: footprint (none) -> Diode_SMD:D_SOD-123
- R1: footprint (none) -> Resistor_SMD:R_1206_3216Metric
- R10, R11, R2, R3, R4, R5, R6, R7, R8, R9: value 4.7 kOM -> 470; footprint (none) -> Resistor_SMD:R_1206_3216Metric
- R12: value 4.7 kOM -> 4.7 K; footprint (none) -> Resistor_SMD:R_1206_3216Metric
Connections:
- net +5V: now also C101.1, J1.A9 (VBUS), J1.B9 (VBUS)
- net GND: now also C101.2, J1.A12 (GND), J1.B12 (GND), SW101.1
- net dc: now also U1.19 (GPIO13/ADC2_CH2); no longer U1.36 (GPIO39/MTCK)
- net reset_tft: now also U1.35 (GPIO38); no longer U1.37 (GPIO40/MTDO)
- net sck: now also U1.18 (GPIO12/ADC2_CH1); no longer U1.7 (GPIO7/ADC1_CH6)
- net sda: now also U1.17 (GPIO11/ADC2_CH0); no longer U1.6 (GPIO6/ADC1_CH5)
- net at R9.1: now also U1.12 (GPIO8/ADC1_CH7); no longer U1.16 (GPIO10/ADC1_CH9)
- net at R1.2: now also U1.36 (GPIO39/MTCK); no longer U1.38 (GPIO41/MTDI)
- net at D101.1 (K): now also U1.20 (GPIO14/ADC2_CH3); no longer U1.19 (GPIO13/ADC2_CH2)
- net at D105.1 (K): now also U1.25 (GPIO19/USB_D-); no longer U1.27 (GPIO21)
- net at D102.1 (K): now also U1.10 (GPIO17/ADC2_CH6); no longer U1.20 (GPIO14/ADC2_CH3)
- net at R11.1: now also U1.16 (GPIO10/ADC1_CH9); no longer U1.18 (GPIO12/ADC2_CH1)
- net at D107.1 (K): now also U1.39 (GPIO42/MTMS); no longer U1.14 (GPIO46)
- net at D103.1 (K): now also U1.11 (GPIO18/ADC2_CH7); no longer U1.10 (GPIO17/ADC2_CH6)
- net at D106.1 (K): now also U1.38 (GPIO41/MTDI); no longer U1.35 (GPIO38)
- net at D104.1 (K): now also U1.27 (GPIO21/RTC); no longer U1.11 (GPIO18/ADC2_CH7)
- net at R7.1: now also U1.6 (GPIO6/ADC1_CH5); no longer U1.12 (GPIO8/ADC1_CH7)
- net at D110.1 (K): now also U1.37 (GPIO40/MTDO); no longer U1.39 (GPIO42/MTMS)
- net at U1.15 (GPIO9/ADC1_CH8): now also R10.1; no longer R8.1
- net key_1: now reaches U1.26 (GPIO20/USB_D+)
- net key_1: now also R13.2
- new net: R13.1, SW101.2
- new net: R8.1, U1.7 (GPIO7/ADC1_CH6)
- no-connect marks 13 -> 14
Other:
- moved on the sheet: D101, D102, D103, D104, D105, D106, D107, D108, D109, D110, LCD1, R1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

Commit message: Update schema and libraries
Parts:
- removed D1, D10, D100, D11, D12, D13, D14, D15, D16, D17, D18, D19, D2, D20, D21, D22, D23, D24, D25, D26, D27, D28, D29, D3, D30, D31, D32, D33, D34, D35, D36, D37, D38, D39, D4, D40, D41, D42, D43, D44, D45, D46, D47, D48, D49, D5, D50, D51, D52, D53, D54, D55, D56, D57, D58, D59, D6, D60, D61, D62, D63, D64, D65, D66, D67, D68, D69, D7, D70, D71, D72, D73, D74, D75, D76, D77, D78, D79, D8, D80, D81, D82, D83, D84, D85, D86, D87, D88, D89, D9, D90, D91, D92, D93, D94, D95, D96, D97, D98, D99: WS2812B, LED_SMD:LED_WS2812B_PLCC4_5.0x5.0mm_P3.2mm, symbol LED:WS2812B
- removed SW1, SW10, SW100, SW11, SW12, SW13, SW14, SW15, SW16, SW17, SW18, SW19, SW2, SW20, SW21, SW22, SW23, SW24, SW25, SW26, SW27, SW28, SW29, SW3, SW30, SW31, SW32, SW33, SW34, SW35, SW36, SW37, SW38, SW39, SW4, SW40, SW41, SW42, SW43, SW44, SW45, SW46, SW47, SW48, SW49, SW5, SW50, SW51, SW52, SW53, SW54, SW55, SW56, SW57, SW58, SW59, SW6, SW60, SW61, SW62, SW63, SW64, SW65, SW66, SW67, SW68, SW69, SW7, SW70, SW71, SW72, SW73, SW74, SW75, SW76, SW77, SW78, SW79, SW8, SW80, SW81, SW82, SW83, SW84, SW85, SW86, SW87, SW88, SW89, SW9, SW90, SW91, SW92, SW93, SW94, SW95, SW96, SW97, SW98, SW99: SW_Push, Button_Switch_Keyboard:SW_Cherry_MX_1.00u_Plate, symbol Switch:SW_Push
- added SW1, SW10, SW100, SW11, SW12, SW13, SW14, SW15, SW16, SW17, SW18, SW19, SW2, SW20, SW21, SW22, SW23, SW24, SW25, SW26, SW27, SW28, SW29, SW3, SW30, SW31, SW32, SW33, SW34, SW35, SW36, SW37, SW38, SW39, SW4, SW40, SW41, SW42, SW43, SW44, SW45, SW46, SW47, SW48, SW49, SW5, SW50, SW51, SW52, SW53, SW54, SW55, SW56, SW57, SW58, SW59, SW6, SW60, SW61, SW62, SW63, SW64, SW65, SW66, SW67, SW68, SW69, SW7, SW70, SW71, SW72, SW73, SW74, SW75, SW76, SW77, SW78, SW79, SW8, SW80, SW81, SW82, SW83, SW84, SW85, SW86, SW87, SW88, SW89, SW9, SW90, SW91, SW92, SW93, SW94, SW95, SW96, SW97, SW98, SW99: ~, Library:SW_Cherry_MX_LED, symbol prj:SW_PUSH_LED
- C1: value 100 n -> C
- renumbered D110 to D1, D105 to D10, D106 to D2, D107 to D3, D109 to D4, D108 to D5, D101 to D6, D102 to D7, D103 to D8, D104 to D9, R8 to R10, R9 to R11, R10 to R12, R11 to R13, R12 to R2, R13 to R3, R2 to R4, R3 to R5, R4 to R6, R5 to R7, R6 to R8, R7 to R9
Connections:
- net +5V: now also SW1.1 (VDD), SW10.1 (VDD), SW100.1 (VDD), SW11.1 (VDD), SW12.1 (VDD), SW13.1 (VDD), SW14.1 (VDD), SW15.1 (VDD), SW16.1 (VDD), SW17.1 (VDD), SW18.1 (VDD), SW19.1 (VDD), SW2.1 (VDD), SW20.1 (VDD), SW21.1 (VDD), SW22.1 (VDD), SW23.1 (VDD), SW24.1 (VDD), SW25.1 (VDD), SW26.1 (VDD), SW27.1 (VDD), SW28.1 (VDD), SW29.1 (VDD), SW3.1 (VDD), SW30.1 (VDD), SW31.1 (VDD), SW32.1 (VDD), SW33.1 (VDD), SW34.1 (VDD), SW35.1 (VDD), SW36.1 (VDD), SW37.1 (VDD), SW38.1 (VDD), SW39.1 (VDD), SW4.1 (VDD), SW40.1 (VDD), SW41.1 (VDD), SW42.1 (VDD), SW43.1 (VDD), SW44.1 (VDD), SW45.1 (VDD), SW46.1 (VDD), SW47.1 (VDD), SW48.1 (VDD), SW49.1 (VDD), SW5.1 (VDD), SW50.1 (VDD), SW51.1 (VDD), SW52.1 (VDD), SW53.1 (VDD), SW54.1 (VDD), SW55.1 (VDD), SW56.1 (VDD), SW57.1 (VDD), SW58.1 (VDD), SW59.1 (VDD), SW6.1 (VDD), SW60.1 (VDD), SW61.1 (VDD), SW62.1 (VDD), SW63.1 (VDD), SW64.1 (VDD), SW65.1 (VDD), SW66.1 (VDD), SW67.1 (VDD), SW68.1 (VDD), SW69.1 (VDD), SW7.1 (VDD), SW70.1 (VDD), SW71.1 (VDD), SW72.1 (VDD), SW73.1 (VDD), SW74.1 (VDD), SW75.1 (VDD), SW76.1 (VDD), SW77.1 (VDD), SW78.1 (VDD), SW79.1 (VDD), SW8.1 (VDD), SW80.1 (VDD), SW81.1 (VDD), SW82.1 (VDD), SW83.1 (VDD), SW84.1 (VDD), SW85.1 (VDD), SW86.1 (VDD), SW87.1 (VDD), SW88.1 (VDD), SW89.1 (VDD), SW9.1 (VDD), SW90.1 (VDD), SW91.1 (VDD), SW92.1 (VDD), SW93.1 (VDD), SW94.1 (VDD), SW95.1 (VDD), SW96.1 (VDD), SW97.1 (VDD), SW98.1 (VDD), SW99.1 (VDD)
- net GND: now also SW1.3 (VSS), SW10.3 (VSS), SW100.3 (VSS), SW11.3 (VSS), SW12.3 (VSS), SW13.3 (VSS), SW14.3 (VSS), SW15.3 (VSS), SW16.3 (VSS), SW17.3 (VSS), SW18.3 (VSS), SW19.3 (VSS), SW2.3 (VSS), SW20.3 (VSS), SW21.3 (VSS), SW22.3 (VSS), SW23.3 (VSS), SW24.3 (VSS), SW25.3 (VSS), SW26.3 (VSS), SW27.3 (VSS), SW28.3 (VSS), SW29.3 (VSS), SW3.3 (VSS), SW30.3 (VSS), SW31.3 (VSS), SW32.3 (VSS), SW33.3 (VSS), SW34.3 (VSS), SW35.3 (VSS), SW36.3 (VSS), SW37.3 (VSS), SW38.3 (VSS), SW39.3 (VSS), SW4.3 (VSS), SW40.3 (VSS), SW41.3 (VSS), SW42.3 (VSS), SW43.3 (VSS), SW44.3 (VSS), SW45.3 (VSS), SW46.3 (VSS), SW47.3 (VSS), SW48.3 (VSS), SW49.3 (VSS), SW5.3 (VSS), SW50.3 (VSS), SW51.3 (VSS), SW52.3 (VSS), SW53.3 (VSS), SW54.3 (VSS), SW55.3 (VSS), SW56.3 (VSS), SW57.3 (VSS), SW58.3 (VSS), SW59.3 (VSS), SW6.3 (VSS), SW60.3 (VSS), SW61.3 (VSS), SW62.3 (VSS), SW63.3 (VSS), SW64.3 (VSS), SW65.3 (VSS), SW66.3 (VSS), SW67.3 (VSS), SW68.3 (VSS), SW69.3 (VSS), SW7.3 (VSS), SW70.3 (VSS), SW71.3 (VSS), SW72.3 (VSS), SW73.3 (VSS), SW74.3 (VSS), SW75.3 (VSS), SW76.3 (VSS), SW77.3 (VSS), SW78.3 (VSS), SW79.3 (VSS), SW8.3 (VSS), SW80.3 (VSS), SW81.3 (VSS), SW82.3 (VSS), SW83.3 (VSS), SW84.3 (VSS), SW85.3 (VSS), SW86.3 (VSS), SW87.3 (VSS), SW88.3 (VSS), SW89.3 (VSS), SW9.3 (VSS), SW90.3 (VSS), SW91.3 (VSS), SW92.3 (VSS), SW93.3 (VSS), SW94.3 (VSS), SW95.3 (VSS), SW96.3 (VSS), SW97.3 (VSS), SW98.3 (VSS), SW99.3 (VSS)
- net cl_1: now also SW1.6 (SW_2), SW10.6 (SW_2), SW2.6 (SW_2), SW3.6 (SW_2), SW4.6 (SW_2), SW5.6 (SW_2), SW6.6 (SW_2), SW7.6 (SW_2), SW8.6 (SW_2), SW9.6 (SW_2)
- net cl_10: now also SW100.6 (SW_2), SW91.6 (SW_2), SW92.6 (SW_2), SW93.6 (SW_2), SW94.6 (SW_2), SW95.6 (SW_2), SW96.6 (SW_2), SW97.6 (SW_2), SW98.6 (SW_2), SW99.6 (SW_2)
- net cl_2: now also SW11.6 (SW_2), SW12.6 (SW_2), SW13.6 (SW_2), SW14.6 (SW_2), SW15.6 (SW_2), SW16.6 (SW_2), SW17.6 (SW_2), SW18.6 (SW_2), SW19.6 (SW_2), SW20.6 (SW_2)
- net cl_3: now also SW21.6 (SW_2), SW22.6 (SW_2), SW23.6 (SW_2), SW24.6 (SW_2), SW25.6 (SW_2), SW26.6 (SW_2), SW27.6 (SW_2), SW28.6 (SW_2), SW29.6 (SW_2), SW30.6 (SW_2)
- net cl_4: now also SW31.6 (SW_2), SW32.6 (SW_2), SW33.6 (SW_2), SW34.6 (SW_2), SW35.6 (SW_2), SW36.6 (SW_2), SW37.6 (SW_2), SW38.6 (SW_2), SW39.6 (SW_2), SW40.6 (SW_2)
- net cl_5: now also SW41.6 (SW_2), SW42.6 (SW_2), SW43.6 (SW_2), SW44.6 (SW_2), SW45.6 (SW_2), SW46.6 (SW_2), SW47.6 (SW_2), SW48.6 (SW_2), SW49.6 (SW_2), SW50.6 (SW_2)
- net cl_6: now also SW51.6 (SW_2), SW52.6 (SW_2), SW53.6 (SW_2), SW54.6 (SW_2), SW55.6 (SW_2), SW56.6 (SW_2), SW57.6 (SW_2), SW58.6 (SW_2), SW59.6 (SW_2), SW60.6 (SW_2)
- net cl_7: now also SW61.6 (SW_2), SW62.6 (SW_2), SW63.6 (SW_2), SW64.6 (SW_2), SW65.6 (SW_2), SW66.6 (SW_2), SW67.6 (SW_2), SW68.6 (SW_2), SW69.6 (SW_2), SW70.6 (SW_2)
- net cl_8: now also SW71.6 (SW_2), SW72.6 (SW_2), SW73.6 (SW_2), SW74.6 (SW_2), SW75.6 (SW_2), SW76.6 (SW_2), SW77.6 (SW_2), SW78.6 (SW_2), SW79.6 (SW_2), SW80.6 (SW_2)
- net cl_9: now also SW81.6 (SW_2), SW82.6 (SW_2), SW83.6 (SW_2), SW84.6 (SW_2), SW85.6 (SW_2), SW86.6 (SW_2), SW87.6 (SW_2), SW88.6 (SW_2), SW89.6 (SW_2), SW90.6 (SW_2)
- net led_1: now also SW2.4 (DIN), SW91.2 (DOUT)
- net led_2: now also SW3.4 (DIN), SW92.2 (DOUT)
- net led_3: now also SW4.4 (DIN), SW93.2 (DOUT)
- net led_4: now also SW5.4 (DIN), SW94.2 (DOUT)
- net led_5: now also SW6.4 (DIN), SW95.2 (DOUT)
- net led_6: now also SW7.4 (DIN), SW96.2 (DOUT)
- net led_7: now also SW8.4 (DIN), SW97.2 (DOUT)
- net led_8: now also SW9.4 (DIN), SW98.2 (DOUT)
- net led_9: now also SW10.4 (DIN), SW99.2 (DOUT)
- net rgb_in: now also SW1.4 (DIN)
- net row_1: now also SW1.5 (SW_1), SW11.5 (SW_1), SW21.5 (SW_1), SW31.5 (SW_1), SW41.5 (SW_1), SW51.5 (SW_1), SW61.5 (SW_1), SW71.5 (SW_1), SW81.5 (SW_1), SW91.5 (SW_1)
- net row_10: now also SW10.5 (SW_1), SW100.5 (SW_1), SW20.5 (SW_1), SW30.5 (SW_1), SW40.5 (SW_1), SW50.5 (SW_1), SW60.5 (SW_1), SW70.5 (SW_1), SW80.5 (SW_1), SW90.5 (SW_1)
- net row_2: now also SW12.5 (SW_1), SW2.5 (SW_1), SW22.5 (SW_1), SW32.5 (SW_1), SW42.5 (SW_1), SW52.5 (SW_1), SW62.5 (SW_1), SW72.5 (SW_1), SW82.5 (SW_1), SW92.5 (SW_1)
- net row_3: now also SW13.5 (SW_1), SW23.5 (SW_1), SW3.5 (SW_1), SW33.5 (SW_1), SW43.5 (SW_1), SW53.5 (SW_1), SW63.5 (SW_1), SW73.5 (SW_1), SW83.5 (SW_1), SW93.5 (SW_1)
- net row_4: now also SW14.5 (SW_1), SW24.5 (SW_1), SW34.5 (SW_1), SW4.5 (SW_1), SW44.5 (SW_1), SW54.5 (SW_1), SW64.5 (SW_1), SW74.5 (SW_1), SW84.5 (SW_1), SW94.5 (SW_1)
- net row_5: now also SW15.5 (SW_1), SW25.5 (SW_1), SW35.5 (SW_1), SW45.5 (SW_1), SW5.5 (SW_1), SW55.5 (SW_1), SW65.5 (SW_1), SW75.5 (SW_1), SW85.5 (SW_1), SW95.5 (SW_1)
- net row_6: now also SW16.5 (SW_1), SW26.5 (SW_1), SW36.5 (SW_1), SW46.5 (SW_1), SW56.5 (SW_1), SW6.5 (SW_1), SW66.5 (SW_1), SW76.5 (SW_1), SW86.5 (SW_1), SW96.5 (SW_1)
- net row_7: now also SW17.5 (SW_1), SW27.5 (SW_1), SW37.5 (SW_1), SW47.5 (SW_1), SW57.5 (SW_1), SW67.5 (SW_1), SW7.5 (SW_1), SW77.5 (SW_1), SW87.5 (SW_1), SW97.5 (SW_1)
- net row_8: now also SW18.5 (SW_1), SW28.5 (SW_1), SW38.5 (SW_1), SW48.5 (SW_1), SW58.5 (SW_1), SW68.5 (SW_1), SW78.5 (SW_1), SW8.5 (SW_1), SW88.5 (SW_1), SW98.5 (SW_1)
- net row_9: now also SW19.5 (SW_1), SW29.5 (SW_1), SW39.5 (SW_1), SW49.5 (SW_1), SW59.5 (SW_1), SW69.5 (SW_1), SW79.5 (SW_1), SW89.5 (SW_1), SW9.5 (SW_1), SW99.5 (SW_1)
- new net: SW85.2 (DOUT), SW95.4 (DIN)
- new net: SW21.2 (DOUT), SW31.4 (DIN)
- new net: SW11.2 (DOUT), SW21.4 (DIN)
- new net: SW62.2 (DOUT), SW72.4 (DIN)
- new net: SW52.2 (DOUT), SW62.4 (DIN)
- new net: SW81.2 (DOUT), SW91.4 (DIN)
- new net: SW84.2 (DOUT), SW94.4 (DIN)
- new net: SW69.2 (DOUT), SW79.4 (DIN)
- new net: SW59.2 (DOUT), SW69.4 (DIN)
- new net: SW75.2 (DOUT), SW85.4 (DIN)
- new net: SW16.2 (DOUT), SW26.4 (DIN)
- new net: SW16.4 (DIN), SW6.2 (DOUT)
- new net: SW63.2 (DOUT), SW73.4 (DIN)
- new net: SW53.2 (DOUT), SW63.4 (DIN)
- new net: SW13.4 (DIN), SW3.2 (DOUT)
- new net: SW23.2 (DOUT), SW33.4 (DIN)
- new net: SW13.2 (DOUT), SW23.4 (DIN)
- new net: SW65.2 (DOUT), SW75.4 (DIN)
- new net: SW55.2 (DOUT), SW65.4 (DIN)
- new net: SW42.2 (DOUT), SW52.4 (DIN)
- new net: SW32.2 (DOUT), SW42.4 (DIN)
- new net: SW83.2 (DOUT), SW93.4 (DIN)
- new net: SW39.2 (DOUT), SW49.4 (DIN)
- new net: SW29.2 (DOUT), SW39.4 (DIN)
- new net: SW18.2 (DOUT), SW28.4 (DIN)
- new net: SW18.4 (DIN), SW8.2 (DOUT)
- new net: SW17.2 (DOUT), SW27.4 (DIN)
- new net: SW17.4 (DIN), SW7.2 (DOUT)
- new net: SW38.2 (DOUT), SW48.4 (DIN)
- new net: SW28.2 (DOUT), SW38.4 (DIN)
- new net: SW71.2 (DOUT), SW81.4 (DIN)
- new net: SW61.2 (DOUT), SW71.4 (DIN)
- new net: SW77.2 (DOUT), SW87.4 (DIN)
- new net: SW67.2 (DOUT), SW77.4 (DIN)
- new net: SW45.2 (DOUT), SW55.4 (DIN)
- new net: SW57.2 (DOUT), SW67.4 (DIN)
- new net: SW31.2 (DOUT), SW41.4 (DIN)
- new net: SW80.2 (DOUT), SW90.4 (DIN)
- new net: SW70.2 (DOUT), SW80.4 (DIN)
- new net: SW86.2 (DOUT), SW96.4 (DIN)
- new net: SW76.2 (DOUT), SW86.4 (DIN)
- new net: SW35.2 (DOUT), SW45.4 (DIN)
- new net: SW88.2 (DOUT), SW98.4 (DIN)
- new net: SW22.2 (DOUT), SW32.4 (DIN)
- new net: SW12.2 (DOUT), SW22.4 (DIN)
- new net: SW33.2 (DOUT), SW43.4 (DIN)
- new net: SW51.2 (DOUT), SW61.4 (DIN)
- new net: SW25.2 (DOUT), SW35.4 (DIN)
- new net: SW15.2 (DOUT), SW25.4 (DIN)
- new net: SW34.2 (DOUT), SW44.4 (DIN)
- new net: SW24.2 (DOUT), SW34.4 (DIN)
- new net: SW14.2 (DOUT), SW24.4 (DIN)
- new net: SW14.4 (DIN), SW4.2 (DOUT)
- new net: SW60.2 (DOUT), SW70.4 (DIN)
- new net: SW37.2 (DOUT), SW47.4 (DIN)
- new net: SW27.2 (DOUT), SW37.4 (DIN)
- new net: SW49.2 (DOUT), SW59.4 (DIN)
- new net: SW56.2 (DOUT), SW66.4 (DIN)
- new net: SW46.2 (DOUT), SW56.4 (DIN)
- new net: SW19.2 (DOUT), SW29.4 (DIN)
- new net: SW78.2 (DOUT), SW88.4 (DIN)
- new net: SW68.2 (DOUT), SW78.4 (DIN)
- new net: SW66.2 (DOUT), SW76.4 (DIN)
- new net: SW100.4 (DIN), SW90.2 (DOUT)
- new net: SW41.2 (DOUT), SW51.4 (DIN)
- new net: SW74.2 (DOUT), SW84.4 (DIN)
- new net: SW64.2 (DOUT), SW74.4 (DIN)
- new net: SW43.2 (DOUT), SW53.4 (DIN)
- new net: SW1.2 (DOUT), SW11.4 (DIN)
- new net: SW15.4 (DIN), SW5.2 (DOUT)
- new net: SW54.2 (DOUT), SW64.4 (DIN)
- new net: SW44.2 (DOUT), SW54.4 (DIN)
- new net: SW73.2 (DOUT), SW83.4 (DIN)
- new net: SW26.2 (DOUT), SW36.4 (DIN)
- new net: SW30.2 (DOUT), SW40.4 (DIN)
- new net: SW20.2 (DOUT), SW30.4 (DIN)
- new net: SW82.2 (DOUT), SW92.4 (DIN)
- new net: SW72.2 (DOUT), SW82.4 (DIN)
- new net: SW50.2 (DOUT), SW60.4 (DIN)
- new net: SW40.2 (DOUT), SW50.4 (DIN)
- new net: SW87.2 (DOUT), SW97.4 (DIN)
- new net: SW19.4 (DIN), SW9.2 (DOUT)
- new net: SW47.2 (DOUT), SW57.4 (DIN)
- new net: SW79.2 (DOUT), SW89.4 (DIN)
- new net: SW48.2 (DOUT), SW58.4 (DIN)
- new net: SW58.2 (DOUT), SW68.4 (DIN)
- new net: SW36.2 (DOUT), SW46.4 (DIN)
- new net: SW89.2 (DOUT), SW99.4 (DIN)
- new net: SW10.2 (DOUT), SW20.4 (DIN)
- new net: SW12.4 (DIN), SW2.2 (DOUT)
Other:
- moved on the sheet: C101, D1, D10, D2, D3, D4, D5, D6, D7, D8, D9, J1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

Commit message: Draft of PCB
Connections:
- net +3V3: now also LCD1.2 (VCC); no longer LCD1.1 (GND)
Changed lines of the file:
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@@
 		(pin "1"
 		)
-		(pin "1"
+		(pin "2"
 		)
 		(pin "7"

Commit message: Add new layout, update schema
Parts:
- added J2: Conn_01x04, Connector_PinSocket_2.54mm:PinSocket_1x04_P2.54mm_Vertical, symbol Connector_Generic:Conn_01x04
- SW1, SW10, SW100, SW11, SW12, SW13, SW14, SW15, SW16, SW17, SW18, SW19, SW2, SW20, SW21, SW22, SW23, SW24, SW25, SW26, SW27, SW28, SW29, SW3, SW30, SW31, SW32, SW33, SW34, SW35, SW36, SW37, SW38, SW39, SW4, SW40, SW41, SW42, SW43, SW44, SW45, SW46, SW47, SW48, SW49, SW5, SW50, SW51, SW52, SW53, SW54, SW55, SW56, SW57, SW58, SW59, SW6, SW60, SW61, SW62, SW63, SW64, SW65, SW66, SW67, SW68, SW69, SW7, SW70, SW71, SW72, SW73, SW74, SW75, SW76, SW77, SW78, SW79, SW8, SW80, SW81, SW82, SW83, SW84, SW85, SW86, SW87, SW88, SW89, SW9, SW90, SW91, SW92, SW93, SW94, SW95, SW96, SW97, SW98, SW99: footprint Library:SW_Cherry_MX_LED -> Library:SW_Cherry_MX_LED_2
Connections:
- net +3V3: now also J2.2 (Pin_2)
- net +5V: now also J2.1 (Pin_1)
- net GND: now also J2.3 (Pin_3), J2.4 (Pin_4)
