File: schema_keyboard_game.kicad_sch (KiCad schematic)
At the start: 233 parts, among them J1 USB_C_Receptacle_PowerOnly_6P, J2 Conn_01x02, J3 Conn_01x03, J4 Conn_01x04, SW101 SW_Push, U1 ESP32-S3-DevKitC

Commit message: Add TTL logic, update schema and pcb, draft
Parts:
- added C102: 100p, Capacitor_SMD:C_1206_3216Metric, symbol Device:C
- added R3, R4, R6: 470, Resistor_SMD:R_1206_3216Metric, symbol Device:R
- added U1: 74AHCT125, Package_DIP:DIP-14_W7.62mm, symbol 74xx:74AHCT125
- renumbered C102 to C103, C103 to C104, R7 to R10, R8 to R11, R9 to R12, R10 to R13, R11 to R14, R12 to R15, R13 to R16, R3 to R5, R4 to R7, R5 to R8, R6 to R9, U1 to U2
Connections:
- net +5V: now also C102.2, R3.1, R4.1, R6.1, U1.14 (VCC)
- net GND: now also C102.1, U1.1, U1.7 (GND)
- net rgb_in: now also U1.2; no longer SW1.4 (DIN)
- new net: R4.2, U1.10, U1.9
- new net: R6.2, U1.12, U1.13
- new net: R3.2, U1.4, U1.5
- new net rgb_in_5V: SW1.4 (DIN), U1.3
- no-connect marks 12 -> 15

Commit message: Schema and PCB, ver 1.5
Parts:
- added C105: 100p, Capacitor_SMD:C_1206_3216Metric, symbol Device:C
- added R17, R18: 4.7 K, Resistor_SMD:R_1206_3216Metric, symbol Device:R
Connections:
- net +3V3: now also R17.2, R18.2
- net GND: now also C105.2
- net key_1: now also C105.1
- net sck: now also R18.1
- net sda: now also R17.1

Commit message: Update USB connection, update values
Parts:
- added R19, R20: 5.1k, Resistor_SMD:R_1206_3216Metric, symbol Device:R
- C1, C10, C100, C103, C104, C11, C12, C13, C14, C15, C16, C17, C18, C19, C2, C20, C21, C22, C23, C24, C25, C26, C27, C28, C29, C3, C30, C31, C32, C33, C34, C35, C36, C37, C38, C39, C4, C40, C41, C42, C43, C44, C45, C46, C47, C48, C49, C5, C50, C51, C52, C53, C54, C55, C56, C57, C58, C59, C6, C60, C61, C62, C63, C64, C65, C66, C67, C68, C69, C7, C70, C71, C72, C73, C74, C75, C76, C77, C78, C79, C8, C80, C81, C82, C83, C84, C85, C86, C87, C88, C89, C9, C90, C91, C92, C93, C94, C95, C96, C97, C98, C99: value C -> 100n
- C101: value 100 nF -> 100n
- D1, D10, D2, D3, D4, D5, D6, D7, D8, D9: value D -> 1N4148
- R1: value 470 OM -> 470
- R3, R4, R6: value 470 -> 5.1k
Connections:
- net GND: now also R19.1, R20.1
- net at J1.A5 (CC1): now also R20.2
- net at J1.B5 (CC2): now also R19.2
- no-connect marks 15 -> 13
