File: schema_2/schema_2.kicad_sch (KiCad schematic)
At the start: 0 parts

Commit message: Straight forward for schema 2
Parts:
- added C1, C10, C100, C11, C12, C13, C14, C15, C16, C17, C18, C19, C2, C20, C21, C22, C23, C24, C25, C26, C27, C28, C29, C3, C30, C31, C32, C33, C34, C35, C36, C37, C38, C39, C4, C40, C41, C42, C43, C44, C45, C46, C47, C48, C49, C5, C50, C51, C52, C53, C54, C55, C56, C57, C58, C59, C6, C60, C61, C62, C63, C64, C65, C66, C67, C68, C69, C7, C70, C71, C72, C73, C74, C75, C76, C77, C78, C79, C8, C80, C81, C82, C83, C84, C85, C86, C87, C88, C89, C9, C90, C91, C92, C93, C94, C95, C96, C97, C98, C99: 100n, symbol Device:C
- added C101: 100n, Capacitor_SMD:C_1206_3216Metric, symbol Device:C
- added C102, C105, C106: 100p, Capacitor_SMD:C_1206_3216Metric, symbol Device:C
- added C103, C104, C107, C108, C109, C110, C111, C112, C113: C, symbol Device:C
- added D1: D_TVS, symbol Device:D_TVS
- added J1: USB_C_Receptacle_PowerOnly_6P, Connector_USB:USB_C_Receptacle_HRO_TYPE-C-31-M-17, symbol Connector:USB_C_Receptacle_PowerOnly_6P
- added LCD1: ST7789_1.3_240x240_LCD_Module, ST7789_1.3_240x240_LCD_Module:ST7789_1.3_240x240_LCD_Module, symbol ST7789_1.3_240x240_LCD_Module:ST7789_1.3_240x240_LCD_Module
- added LS1: Speaker, symbol Device:Speaker
- added R1, R10, R8, R9: R, symbol Device:R
- added R19, R20, R3, R4, R7: 5.1k, Resistor_SMD:R_1206_3216Metric, symbol Device:R
- added R2: 4.7 K, Resistor_SMD:R_1206_3216Metric, symbol Device:R
- added R5, R6: 470, Resistor_SMD:R_1206_3216Metric, symbol Device:R
- added SW1, SW10, SW100, SW11, SW12, SW13, SW14, SW15, SW16, SW17, SW18, SW19, SW2, SW20, SW21, SW22, SW23, SW24, SW25, SW26, SW27, SW28, SW29, SW3, SW30, SW31, SW32, SW33, SW34, SW35, SW36, SW37, SW38, SW39, SW4, SW40, SW41, SW42, SW43, SW44, SW45, SW46, SW47, SW48, SW49, SW5, SW50, SW51, SW52, SW53, SW54, SW55, SW56, SW57, SW58, SW59, SW6, SW60, SW61, SW62, SW63, SW64, SW65, SW66, SW67, SW68, SW69, SW7, SW70, SW71, SW72, SW73, SW74, SW75, SW76, SW77, SW78, SW79, SW8, SW80, SW81, SW82, SW83, SW84, SW85, SW86, SW87, SW88, SW89, SW9, SW90, SW91, SW92, SW93, SW94, SW95, SW96, SW97, SW98, SW99: (no value), sw_led:SW_MX_1u_SK6812MINI-E_ROTATE, symbol sw_led:sw_led
- added SW101, SW102: SW_Push, Button_Switch_THT:SW_PUSH_6mm, symbol Switch:SW_Push
- added U1: STM32G070RBTx, Package_QFP:LQFP-64_10x10mm_P0.5mm, symbol MCU_ST_STM32G0:STM32G070RBTx
- added U2: 74AHCT125, Package_DIP:DIP-14_W7.62mm, symbol 74xx:74AHCT125
- added U3: AP2112K-3.3, Package_TO_SOT_SMD:SOT-23-5, symbol Regulator_Linear:AP2112K-3.3
- added U4: W25Q128JVS, Package_SO:SOIC-8_5.3x5.3mm_P1.27mm, symbol Memory_Flash:W25Q128JVS
- added U5: MAX98357A, Package_DFN_QFN:TQFN-16-1EP_3x3mm_P0.5mm_EP1.23x1.23mm, symbol Audio:MAX98357A
- added Y1: ASCO, Oscillator:Oscillator_SMD_Abracon_ASCO-4Pin_1.6x1.2mm, symbol Oscillator:ASCO
Connections:
- new net: SW52.2 (DOUT), SW54.4 (DIN)
- new net: SW50.2 (DOUT), SW52.4 (DIN)
- new net: SW48.2 (DOUT), SW50.4 (DIN)
- new net: SW73.2 (DOUT), SW75.4 (DIN)
- new net: SW71.2 (DOUT), SW73.4 (DIN)
- new net: SW19.2 (DOUT), SW20.4 (DIN)
- new net: SW18.2 (DOUT), SW19.4 (DIN)
- new net: SW17.2 (DOUT), SW18.4 (DIN)
- new net: SW57.2 (DOUT), SW59.4 (DIN)
- new net: SW55.2 (DOUT), SW57.4 (DIN)
- new net: SW44.2 (DOUT), SW46.4 (DIN)
- new net: SW42.2 (DOUT), SW44.4 (DIN)
- new net: LCD1.7 (BLK), R2.2
- new net: SW25.2 (DOUT), SW27.4 (DIN)
- new net: SW23.2 (DOUT), SW25.4 (DIN)
- new net: SW54.2 (DOUT), SW56.4 (DIN)
- new net: SW100.4 (DIN), SW98.2 (DOUT)
- new net: SW96.2 (DOUT), SW98.4 (DIN)
- new net: SW8.2 (DOUT), SW9.4 (DIN)
- new net: SW7.2 (DOUT), SW8.4 (DIN)
- new net: SW84.2 (DOUT), SW86.4 (DIN)
- new net: SW82.2 (DOUT), SW84.4 (DIN)
- new net: R1.2, U3.3 (EN)
- new net: SW49.2 (DOUT), SW51.4 (DIN)
- new net: SW47.2 (DOUT), SW49.4 (DIN)
- new net: SW36.2 (DOUT), SW38.4 (DIN)
- new net: SW34.2 (DOUT), SW36.4 (DIN)
- new net: SW93.2 (DOUT), SW95.4 (DIN)
- new net: SW91.2 (DOUT), SW93.4 (DIN)
- new net: SW6.2 (DOUT), SW7.4 (DIN)
- new net: SW95.2 (DOUT), SW97.4 (DIN)
- new net: SW85.2 (DOUT), SW87.4 (DIN)
- new net: SW83.2 (DOUT), SW85.4 (DIN)
- new net: SW38.2 (DOUT), SW40.4 (DIN)
- new net: SW33.2 (DOUT), SW35.4 (DIN)
- new net: SW31.2 (DOUT), SW33.4 (DIN)
- new net: SW10.4 (DIN), SW9.2 (DOUT)
- new net: SW74.2 (DOUT), SW76.4 (DIN)
- new net: SW72.2 (DOUT), SW74.4 (DIN)
- new net: SW21.2 (DOUT), SW23.4 (DIN)
- new net: R9.2, U4.7 (~{HOLD}/~{RESET}/IO_{3})
- new net: SW3.2 (DOUT), SW4.4 (DIN)
- new net: SW2.2 (DOUT), SW3.4 (DIN)
- new net: SW88.2 (DOUT), SW90.4 (DIN)
- new net: SW86.2 (DOUT), SW88.4 (DIN)
- new net: SW63.2 (DOUT), SW65.4 (DIN)
- new net: SW61.2 (DOUT), SW63.4 (DIN)
- new net: SW12.2 (DOUT), SW13.4 (DIN)
- new net: SW11.2 (DOUT), SW12.4 (DIN)
- new net: SW46.2 (DOUT), SW48.4 (DIN)
- new net: SW28.2 (DOUT), SW30.4 (DIN)
- new net: SW26.2 (DOUT), SW28.4 (DIN)
- new net: SW37.2 (DOUT), SW39.4 (DIN)
- new net: SW35.2 (DOUT), SW37.4 (DIN)
- new net: SW13.2 (DOUT), SW14.4 (DIN)
- new net: SW90.2 (DOUT), SW92.4 (DIN)
- new net: SW58.2 (DOUT), SW60.4 (DIN)
- new net: R5.1, SW101.2
- new net: SW43.2 (DOUT), SW45.4 (DIN)
- new net: SW41.2 (DOUT), SW43.4 (DIN)
- new net: SW45.2 (DOUT), SW47.4 (DIN)
- new net: SW5.2 (DOUT), SW6.4 (DIN)
- new net: SW4.2 (DOUT), SW5.4 (DIN)
- new net: SW70.2 (DOUT), SW72.4 (DIN)
- new net: SW68.2 (DOUT), SW70.4 (DIN)
- new net: SW16.2 (DOUT), SW17.4 (DIN)
- new net: SW15.2 (DOUT), SW16.4 (DIN)
- new net: R3.2, U2.4, U2.5
- new net: SW32.2 (DOUT), SW34.4 (DIN)
- new net: R4.2, U2.10, U2.9
- new net: SW22.2 (DOUT), SW24.4 (DIN)
- new net: SW24.2 (DOUT), SW26.4 (DIN)
- new net: SW78.2 (DOUT), SW80.4 (DIN)
- new net: SW76.2 (DOUT), SW78.4 (DIN)
- new net: SW29.2 (DOUT), SW31.4 (DIN)
- new net: SW27.2 (DOUT), SW29.4 (DIN)
- new net: SW64.2 (DOUT), SW66.4 (DIN)
- new net: SW62.2 (DOUT), SW64.4 (DIN)
- new net: SW77.2 (DOUT), SW79.4 (DIN)
- new net: SW75.2 (DOUT), SW77.4 (DIN)
- new net: SW66.2 (DOUT), SW68.4 (DIN)
- new net: R8.2, Y1.1 (Tri-State)
- new net: SW14.2 (DOUT), SW15.4 (DIN)
- new net: SW56.2 (DOUT), SW58.4 (DIN)
- new net: SW97.2 (DOUT), SW99.4 (DIN)
- new net: SW53.2 (DOUT), SW55.4 (DIN)
- new net: SW1.2 (DOUT), SW2.4 (DIN)
- new net: SW92.2 (DOUT), SW94.4 (DIN)
- new net: SW51.2 (DOUT), SW53.4 (DIN)
- new net: SW89.2 (DOUT), SW91.4 (DIN)
- new net: SW87.2 (DOUT), SW89.4 (DIN)
- new net: R10.2, U4.3 (~{WP}/IO_{2})
- new net: J1.A5 (CC1), R20.2
- new net: J1.B5 (CC2), R19.2
- new net: SW67.2 (DOUT), SW69.4 (DIN)
- new net: SW65.2 (DOUT), SW67.4 (DIN)
- new net: SW94.2 (DOUT), SW96.4 (DIN)
- new net: LS1.1, U5.9 (OUTP)
- new net: LS1.2, U5.10 (OUTN)
- new net: SW30.2 (DOUT), SW32.4 (DIN)
- new net: R7.2, U2.12, U2.13
- new net: R6.1, SW102.2
- new net: SW81.2 (DOUT), SW83.4 (DIN)
- new net: SW69.2 (DOUT), SW71.4 (DIN)
- new net +3V3: C103.1, C107.1, C108.1, C109.1, C110.1, C111.1, LCD1.2 (VCC), R10.1, R2.1, R8.1, R9.1, U1.8 (VDD), U3.5 (VOUT), U4.8 (VCC), Y1.4 (VDD)
- new net +5V: C1.1, C10.1, C100.1, C101.1, C102.2, C104.1, C11.1, C112.1, C113.1, C12.1, C13.1, C14.1, C15.1, C16.1, C17.1, C18.1, C19.1, C2.1, C20.1, C21.1, C22.1, C23.1, C24.1, C25.1, C26.1, C27.1, C28.1, C29.1, C3.1, C30.1, C31.1, C32.1, C33.1, C34.1, C35.1, C36.1, C37.1, C38.1, C39.1, C4.1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
- new net GND: C1.2, C10.2, C100.2, C101.2, C102.1, C103.2, C104.2, C105.2, C106.2, C107.2, C108.2, C109.2, C11.2, C110.2, C111.2, C112.2, C113.2, C12.2, C13.2, C14.2, C15.2, C16.2, C17.2, C18.2, C19.2, C2.2, C20.2, C21.2, C22.2, C23.2, C24.2, C25.2, C26.2, C27.2, C28.2, C29.2, C3.2, C30.2, C31.2, C32.2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
- new net audio_bclk: U5.16 (BCLK)
- new net audio_din: U5.1 (DIN)
- new net audio_lrclk: U5.14 (LRCLK)
- new net audio_mode: U5.4 (~{SD_MODE})
- new net col_1: SW1.6 (SW_2)
- new net col_10: SW10.6 (SW_2), SW100.6 (SW_2), SW20.6 (SW_2), SW39.6 (SW_2), SW40.6 (SW_2), SW59.6 (SW_2), SW60.6 (SW_2), SW79.6 (SW_2), SW80.6 (SW_2), SW99.6 (SW_2)
- new net col_2: SW2.6 (SW_2)
- new net col_3: SW3.6 (SW_2)
- new net col_4: SW4.6 (SW_2)
- new net col_5: SW5.6 (SW_2)
- new net col_6: SW6.6 (SW_2)
- new net col_7: SW7.6 (SW_2)
- new net col_8: SW8.6 (SW_2)
- new net col_9: SW9.6 (SW_2)
- new net dc_lcd: LCD1.6 (DC)
- new net key_1: C105.1, R5.2
- new net key_2: C106.1, R6.2
- new net led_out_1: SW10.2 (DOUT), SW11.4 (DIN)
- new net led_out_2: SW20.2 (DOUT), SW21.4 (DIN)
- new net led_out_3: SW22.4 (DIN), SW39.2 (DOUT)
- new net led_out_4: SW40.2 (DOUT), SW41.4 (DIN)
- new net led_out_5: SW42.4 (DIN), SW59.2 (DOUT)
- new net led_out_6: SW60.2 (DOUT), SW61.4 (DIN)
- new net led_out_7: SW62.4 (DIN), SW79.2 (DOUT)
- new net led_out_8: SW80.2 (DOUT), SW81.4 (DIN)
- new net led_out_9: SW82.4 (DIN), SW99.2 (DOUT)
- new net mcu_clk: Y1.3 (OUT)
- new net reset_lcd: LCD1.5 (RES)
- new net rgb_data_3V: U2.2
- new net rgb_data_5V: SW1.4 (DIN), U2.3
- new net row_1: SW1.5 (SW_1), SW10.5 (SW_1), SW2.5 (SW_1), SW3.5 (SW_1), SW4.5 (SW_1), SW5.5 (SW_1), SW6.5 (SW_1), SW7.5 (SW_1), SW8.5 (SW_1), SW9.5 (SW_1)
- new net spi_clk: LCD1.3 (SCK)
- new net spi_data: LCD1.4 (SDA)
- new net spi_mem_clk: U4.6 (CLK)
- new net spi_mem_cs: U4.1 (~{CS})
- new net spi_mem_miso: U4.2 (DO/IO_{1})
- new net spi_mem_mosi: U4.5 (DI/IO_{0})
- no-connect marks 0 -> 5
Other:
- note added: "5V -> 3.3V"
- note added: "Oscillator"
- note added: "SPI memory"
- note added: "USB"

Commit message: 26.10.2026
Parts:
- added C114: 10u, symbol Device:C
- added C115: 100n, Capacitor_SMD:C_1206_3216Metric, symbol Device:C
- added D10, D100, D101, D11, D12, D13, D14, D15, D16, D17, D18, D19, D2, D20, D21, D22, D23, D24, D25, D26, D27, D28, D29, D3, D30, D31, D32, D33, D34, D35, D36, D37, D38, D39, D4, D40, D41, D42, D43, D44, D45, D46, D47, D48, D49, D5, D50, D51, D52, D53, D54, D55, D56, D57, D58, D59, D6, D60, D61, D62, D63, D64, D65, D66, D67, D68, D69, D7, D70, D71, D72, D73, D74, D75, D76, D77, D78, D79, D8, D80, D81, D82, D83, D84, D85, D86, D87, D88, D89, D9, D90, D91, D92, D93, D94, D95, D96, D97, D98, D99: SM4007PL, Diode_SMD:D_SOD-123F, symbol Device:D
- added J2: Conn_01x03_Pin, Connector_PinHeader_2.54mm:PinHeader_1x03_P2.54mm_Vertical, symbol Connector:Conn_01x03_Pin
- added R11: 1k, Resistor_SMD:R_1206_3216Metric, symbol Device:R
- added R12, R13, R14: 10k, Resistor_SMD:R_1206_3216Metric, symbol Device:R
- added SW103, SW104: SK12D07VG3, Button_Switch_THT:SW_Slide_SPDT_Angled_CK_OS102011MA1Q, symbol Switch:SW_SPDT
- added SW105: SW_Push, Button_Switch_THT:SW_PUSH_6mm, symbol Switch:SW_Push
- added U6: WEMOS_D1_mini, RF_Module:WEMOS_D1_mini_light, symbol RF_Module:WEMOS_D1_mini
- C103, C104: value C -> 1u
- C105, C106: value 100p -> 100n
- C107: value C -> 4.7u
- C108, C109, C111: value C -> 100n
- C110: value C -> 10u
- D1: value D_TVS -> H5VL10B; footprint (none) -> Diode_SMD:D_SOD-882
- R5, R6: value 470 -> 1k
Connections:
- net +3V3: now also C114.1, J2.2 (Pin_2), R12.2, R13.2, R14.2
- net +5V: now also SW103.1 (A), SW104.2 (B); no longer C101.1, D1.2 (A2), J1.A9 (VBUS), J1.B9 (VBUS)
- net GND: now also C114.2, C115.2, J2.3 (Pin_3), SW105.1, U6.10 (GND)
- net col_1: now also D12.1 (K), D13.1 (K), D14.1 (K), D15.1 (K), D16.1 (K), D17.1 (K), D18.1 (K), D19.1 (K), D2.1 (K), D20.1 (K); no longer SW1.6 (SW_2)
- net col_10: now also D100.1 (K), D101.1 (K), D11.1 (K), D93.1 (K), D94.1 (K), D95.1 (K), D96.1 (K), D97.1 (K), D98.1 (K), D99.1 (K); no longer SW10.6 (SW_2), SW100.6 (SW_2), SW20.6 (SW_2), SW39.6 (SW_2), SW40.6 (SW_2), SW59.6 (SW_2), SW60.6 (SW_2), SW79.6 (SW_2), SW80.6 (SW_2), SW99.6 (SW_2)
- net col_2: now also D3.1 (K); no longer SW2.6 (SW_2)
- net col_3: now also D30.1 (K), D31.1 (K), D32.1 (K), D33.1 (K), D34.1 (K), D35.1 (K), D36.1 (K), D37.1 (K), D38.1 (K), D4.1 (K); no longer SW3.6 (SW_2)
- net col_4: now also D39.1 (K), D40.1 (K), D41.1 (K), D42.1 (K), D43.1 (K), D44.1 (K), D45.1 (K), D46.1 (K), D47.1 (K), D5.1 (K); no longer SW4.6 (SW_2)
- net col_5: now also D48.1 (K), D49.1 (K), D50.1 (K), D51.1 (K), D52.1 (K), D53.1 (K), D54.1 (K), D55.1 (K), D56.1 (K), D6.1 (K); no longer SW5.6 (SW_2)
- net col_6: now also D57.1 (K), D58.1 (K), D59.1 (K), D60.1 (K), D61.1 (K), D62.1 (K), D63.1 (K), D64.1 (K), D65.1 (K), D7.1 (K); no longer SW6.6 (SW_2)
- net col_7: now also D66.1 (K), D67.1 (K), D68.1 (K), D69.1 (K), D70.1 (K), D71.1 (K), D72.1 (K), D73.1 (K), D74.1 (K), D8.1 (K); no longer SW7.6 (SW_2)
- net col_8: now also D75.1 (K), D76.1 (K), D77.1 (K), D78.1 (K), D79.1 (K), D80.1 (K), D81.1 (K), D82.1 (K), D83.1 (K), D9.1 (K); no longer SW8.6 (SW_2)
- net col_9: now also D10.1 (K), D84.1 (K), D85.1 (K), D86.1 (K), D87.1 (K), D88.1 (K), D89.1 (K), D90.1 (K), D91.1 (K), D92.1 (K); no longer SW9.6 (SW_2)
- net key_1: now also R13.1
- net key_2: now also R14.1
- net row_6: now reaches SW52.5 (SW_1)
- net row_6: now also SW42.5 (SW_1), SW44.5 (SW_1), SW46.5 (SW_1), SW48.5 (SW_1), SW50.5 (SW_1), SW54.5 (SW_1), SW56.5 (SW_1), SW58.5 (SW_1), SW60.5 (SW_1)
- net at SW52.6 (SW_2): now also D61.2 (A)
- net at SW50.6 (SW_2): now also D52.2 (A)
- net row_7: now reaches SW73.5 (SW_1)
- net row_7: now also SW61.5 (SW_1), SW63.5 (SW_1), SW65.5 (SW_1), SW67.5 (SW_1), SW69.5 (SW_1), SW71.5 (SW_1), SW75.5 (SW_1), SW77.5 (SW_1), SW79.5 (SW_1)
- net at SW73.6 (SW_2): now also D71.2 (A)
- net row_2: now reaches SW20.5 (SW_1)
- net row_2: now also SW11.5 (SW_1), SW12.5 (SW_1), SW13.5 (SW_1), SW14.5 (SW_1), SW15.5 (SW_1), SW16.5 (SW_1), SW17.5 (SW_1), SW18.5 (SW_1), SW19.5 (SW_1)
- net at SW18.6 (SW_2): now also D75.2 (A)
- net stm32_reset: now reaches U1.12 (NRST)
- net stm32_reset: now also C115.1, R11.2, R12.1
- net row_5: now reaches SW57.5 (SW_1)
- net row_5: now also SW41.5 (SW_1), SW43.5 (SW_1), SW45.5 (SW_1), SW47.5 (SW_1), SW49.5 (SW_1), SW51.5 (SW_1), SW53.5 (SW_1), SW55.5 (SW_1), SW59.5 (SW_1)
- net at SW57.6 (SW_2): now also D87.2 (A)
- net at SW44.6 (SW_2): now also D25.2 (A)
- net at SW19.6 (SW_2): now also D84.2 (A)
- net row_3: now reaches SW25.5 (SW_1)
- net row_3: now also SW21.5 (SW_1), SW23.5 (SW_1), SW27.5 (SW_1), SW29.5 (SW_1), SW31.5 (SW_1), SW33.5 (SW_1), SW35.5 (SW_1), SW37.5 (SW_1), SW39.5 (SW_1)
- net at SW25.6 (SW_2): now also D31.2 (A)
- net at SW54.6 (SW_2): now also D70.2 (A)
- net row_10: now reaches SW98.5 (SW_1)
- net row_10: now also SW100.5 (SW_1), SW82.5 (SW_1), SW84.5 (SW_1), SW86.5 (SW_1), SW88.5 (SW_1), SW90.5 (SW_1), SW92.5 (SW_1), SW94.5 (SW_1), SW96.5 (SW_1)
- net at SW98.6 (SW_2): now also D92.2 (A)
- net at SW84.6 (SW_2): now also D29.2 (A)
- net at SW49.6 (SW_2): now also D51.2 (A)
- net row_4: now reaches SW36.5 (SW_1)
- net row_4: now also SW22.5 (SW_1), SW24.5 (SW_1), SW26.5 (SW_1), SW28.5 (SW_1), SW30.5 (SW_1), SW32.5 (SW_1), SW34.5 (SW_1), SW38.5 (SW_1), SW40.5 (SW_1)
- net at SW36.6 (SW_2): now also D77.2 (A)
- net row_9: now reaches SW93.5 (SW_1)
- net row_9: now also SW81.5 (SW_1), SW83.5 (SW_1), SW85.5 (SW_1), SW87.5 (SW_1), SW89.5 (SW_1), SW91.5 (SW_1), SW95.5 (SW_1), SW97.5 (SW_1), SW99.5 (SW_1)
- net at SW93.6 (SW_2): now also D73.2 (A)
- net at SW95.6 (SW_2): now also D82.2 (A)
- net at SW85.6 (SW_2): now also D37.2 (A)
- net at SW42.6 (SW_2): now also D16.2 (A)
- net at SW33.6 (SW_2): now also D67.2 (A)
- net row_8: now reaches SW74.5 (SW_1)
- net row_8: now also SW62.5 (SW_1), SW64.5 (SW_1), SW66.5 (SW_1), SW68.5 (SW_1), SW70.5 (SW_1), SW72.5 (SW_1), SW76.5 (SW_1), SW78.5 (SW_1), SW80.5 (SW_1)
- net at SW74.6 (SW_2): now also D72.2 (A)
- net at SW21.6 (SW_2): now also D13.2 (A)
- net at SW88.6 (SW_2): now also D47.2 (A)
- net at SW63.6 (SW_2): now also D26.2 (A)
- net at SW12.6 (SW_2): now also D21.2 (A)
- net at SW46.6 (SW_2): now also D34.2 (A)
- net at SW28.6 (SW_2): now also D41.2 (A)
- net at SW37.6 (SW_2): now also D85.2 (A)
- net at SW82.6 (SW_2): now also D20.2 (A)
- net at SW13.6 (SW_2): now also D30.2 (A)
- net at SW90.6 (SW_2): now also D56.2 (A)
- net at SW43.6 (SW_2): now also D24.2 (A)
- net at SW47.6 (SW_2): now also D42.2 (A)
- net at SW41.6 (SW_2): now also D15.2 (A)
- net at SW70.6 (SW_2): now also D54.2 (A)
- net at SW86.6 (SW_2): now also D38.2 (A)
- net at SW16.6 (SW_2): now also D57.2 (A)
- net at SW35.6 (SW_2): now also D76.2 (A)
- net at SW34.6 (SW_2): now also D68.2 (A)
- net at SW22.6 (SW_2): now also D14.2 (A)
- net at SW72.6 (SW_2): now also D63.2 (A)
- net at SW38.6 (SW_2): now also D86.2 (A)
- net at SW24.6 (SW_2): now also D23.2 (A)
- net at SW78.6 (SW_2): now also D90.2 (A)
- net at SW11.6 (SW_2): now also D12.2 (A)
- net at SW26.6 (SW_2): now also D32.2 (A)
- net at SW29.6 (SW_2): now also D49.2 (A)
- net at SW64.6 (SW_2): now also D27.2 (A)
- net at SW77.6 (SW_2): now also D89.2 (A)
- net at SW61.6 (SW_2): now also D17.2 (A)
- net at SW68.6 (SW_2): now also D45.2 (A)
- net at SW14.6 (SW_2): now also D39.2 (A)
- net at SW31.6 (SW_2): now also D58.2 (A)
- net at SW58.6 (SW_2): now also D88.2 (A)
- net at SW55.6 (SW_2): now also D78.2 (A)
- net at SW15.6 (SW_2): now also D48.2 (A)
- net at SW27.6 (SW_2): now also D40.2 (A)
- net at SW92.6 (SW_2): now also D65.2 (A)
- net at SW51.6 (SW_2): now also D60.2 (A)
- net at SW89.6 (SW_2): now also D55.2 (A)
- net at SW56.6 (SW_2): now also D79.2 (A)
- net at SW17.6 (SW_2): now also D66.2 (A)
- net at SW67.6 (SW_2): now also D44.2 (A)
- net at SW94.6 (SW_2): now also D74.2 (A)
- net at SW53.6 (SW_2): now also D69.2 (A)
- net at SW30.6 (SW_2): now also D50.2 (A)
- net at SW75.6 (SW_2): now also D80.2 (A)
- net at SW76.6 (SW_2): now also D81.2 (A)
- net at SW96.6 (SW_2): now also D83.2 (A)
- net at SW65.6 (SW_2): now also D35.2 (A)
- net at SW91.6 (SW_2): now also D64.2 (A)
- net at SW66.6 (SW_2): now also D36.2 (A)
- net at SW97.6 (SW_2): now also D91.2 (A)
- net at SW23.6 (SW_2): now also D22.2 (A)
- net at SW87.6 (SW_2): now also D46.2 (A)
- net at SW48.6 (SW_2): now also D43.2 (A)
- net at SW83.6 (SW_2): now also D28.2 (A)
- net at SW81.6 (SW_2): now also D19.2 (A)
- net at SW32.6 (SW_2): now also D59.2 (A)
- net at SW62.6 (SW_2): now also D18.2 (A)
- net at SW45.6 (SW_2): now also D33.2 (A)
- net at SW69.6 (SW_2): now also D53.2 (A)
- net at SW71.6 (SW_2): now also D62.2 (A)
- new net: R11.1, SW105.2
- new net: D93.2 (A), SW20.6 (SW_2)
- new net: D7.2 (A), SW6.6 (SW_2)
- new net: D9.2 (A), SW8.6 (SW_2)
- new net: D95.2 (A), SW40.6 (SW_2)
- new net: D11.2 (A), SW10.6 (SW_2)
- new net: D8.2 (A), SW7.6 (SW_2)
- new net: D10.2 (A), SW9.6 (SW_2)
- new net: D4.2 (A), SW3.6 (SW_2)
- new net: SW104.1 (A), U6.9 (5V)
- new net: D97.2 (A), SW60.6 (SW_2)
- new net: D6.2 (A), SW5.6 (SW_2)
- new net: D98.2 (A), SW79.6 (SW_2)
- new net: D101.2 (A), SW100.6 (SW_2)
- new net: D5.2 (A), SW4.6 (SW_2)
- new net: D94.2 (A), SW39.6 (SW_2)
- new net: D96.2 (A), SW59.6 (SW_2)
- new net: D2.2 (A), SW1.6 (SW_2)
- new net: D99.2 (A), SW80.6 (SW_2)
- new net: D100.2 (A), SW99.6 (SW_2)
- new net: D3.2 (A), SW2.6 (SW_2)
- new net +5VD: C101.1, D1.2 (A2), J1.A9 (VBUS), J1.B9 (VBUS), J2.1 (Pin_1), SW103.2 (B)
- no-connect marks 5 -> 9
Other:
- note added: "5V switch"
- note added: "Audio"
- note added: "Buffer, 3.3V -> 5V"
- note added: "Power pins"
- note added: "Service buttons"
- moved on the sheet: C103, C104, C106, C107, C108, R1, R6, SW102, U1, U3

Commit message: 27.10.2026
Parts:
- added J3: Conn_01x04_Pin, Connector_PinHeader_2.54mm:PinHeader_1x04_P2.54mm_Vertical, symbol Connector:Conn_01x04_Pin
- added R15, R16, R17, R18, R21, R22, R23, R24, R25: 22, symbol Device:R
- C112: value C -> 100n
- C113: value C -> 10u
- R10, R8, R9: value R -> 10k
- Y1: value ASCO -> SX3M8.000M20F30TNN
Connections:
- net +3V3: now also J3.3 (Pin_3)
- net GND: now also J3.4 (Pin_4)
- net audio_bclk: now also U1.40 (PD8), R23.1; no longer U5.16 (BCLK)
- net audio_din: now also U1.44 (PA12), R22.1; no longer U5.1 (DIN)
- net audio_lrclk: now also U1.47 (PA15), R24.1; no longer U5.14 (LRCLK)
- net audio_mode: now also U1.43 (PA11)
- net mcu_clk: now also U1.10 (PF0), R25.2; no longer Y1.3 (OUT)
- net spi_mem_clk: now also U1.33 (PB13), R17.1; no longer U4.6 (CLK)
- net spi_mem_cs: now also U1.36 (PA8)
- net spi_mem_miso: now also U1.34 (PB14), R18.1; no longer U4.2 (DO/IO_{1})
- net spi_mem_mosi: now also U1.35 (PB15), R21.1; no longer U4.5 (DI/IO_{0})
- net esp_uart_rx: now reaches U1.37 (PA9)
- net esp_uart_rx: now also U6.15 (RX)
- net esp_uart_tx: now reaches U1.42 (PA10)
- net esp_uart_tx: now also U6.16 (TX)
- net swdio: now reaches U1.45 (PA13)
- net swdio: now also R15.2
- net swclk: now reaches U1.46 (PA14)
- net swclk: now also R16.2
- new net: R23.2, U5.16 (BCLK)
- new net: R18.2, U4.2 (DO/IO_{1})
- new net: R21.2, U4.5 (DI/IO_{0})
- new net: R25.1, Y1.3 (OUT)
- new net: J3.1 (Pin_1), R15.1
- new net: J3.2 (Pin_2), R16.1
- new net: R24.2, U5.14 (LRCLK)
- new net: R22.2, U5.1 (DIN)
- new net: R17.2, U4.6 (CLK)
Other:
- note added: "220 ohm for every row and column GPIO"
- note added: "Debug STM32"
- moved on the sheet: C112, C113, LS1, R10, R9, SW104, U5, U6

Commit message: Change +5V poser supply symbols
Connections:
- net +5V: no longer C1.1, C10.1, C100.1, C11.1, C12.1, C13.1, C14.1, C15.1, C16.1, C17.1, C18.1, C19.1, C2.1, C20.1, C21.1, C22.1, C23.1, C24.1, C25.1, C26.1, C27.1, C28.1, C29.1, C3.1, C30.1, C31.1, C32.1, C33.1, C34.1, C35.1, C36.1, C37.1, C38.1, C39.1, C4.1, C40.1, C41.1, C42.1, C43.1, C44.1, C45.1, C46.1, C47.1, C48.1, C49.1, C5.1, C50.1, C51.1, C52.1, C53.1, C54.1, C55.1, C56.1, C57.1, C58.1, C59.1, C6.1, C60.1, C61.1, C62.1, C63.1, C64.1, C65.1, C66.1, C67.1, C68.1, C69.1, C7.1, C70.1, C71.1, C72.1, C73.1, C74.1, C75.1, C76.1, C77.1, C78.1, C79.1, C8.1, C80.1, C81.1, C82.1, C83.1, C84.1, C85.1, C86.1, C87.1, C88.1, C89.1, C9.1, C90.1, C91.1, C92.1, C93.1, C94.1, C95.1, C96.1, C97.1, C98.1, C99.1, SW1.1 (VDD), SW10.1 (VDD), SW100.1 (VDD), SW104.2 (B), SW11.1 (VDD), SW12.1 (VDD), SW13.1 (VDD), SW14.1 (VDD), SW15.1 (VDD), SW16.1 (VDD), SW17.1 (VDD), SW18.1 (VDD), SW19.1 (VDD), SW2.1 (VDD), SW20.1 (VDD), SW21.1 (VDD), SW22.1 (VDD), SW23.1 (VDD), SW24.1 (VDD), SW25.1 (VDD), SW26.1 (VDD), SW27.1 (VDD), SW28.1 (VDD), SW29.1 (VDD), SW3.1 (VDD), SW30.1 (VDD), SW31.1 (VDD), SW32.1 (VDD), SW33.1 (VDD), SW34.1 (VDD), SW35.1 (VDD), SW36.1 (VDD), SW37.1 (VDD), SW38.1 (VDD), SW39.1 (VDD), SW4.1 (VDD), SW40.1 (VDD), SW41.1 (VDD), SW42.1 (VDD), SW43.1 (VDD), SW44.1 (VDD), SW45.1 (VDD), SW46.1 (VDD), SW47.1 (VDD), SW48.1 (VDD), SW49.1 (VDD), SW5.1 (VDD), SW50.1 (VDD), SW51.1 (VDD), SW52.1 (VDD), SW53.1 (VDD), SW54.1 (VDD), SW55.1 (VDD), SW56.1 (VDD), SW57.1 (VDD), SW58.1 (VDD), SW59.1 (VDD), SW6.1 (VDD), SW60.1 (VDD), SW61.1 (VDD), SW62.1 (VDD), SW63.1 (VDD), SW64.1 (VDD), SW65.1 (VDD), SW66.1 (VDD), SW67.1 (VDD), SW68.1 (VDD), SW69.1 (VDD), SW7.1 (VDD), SW70.1 (VDD), SW71.1 (VDD), SW72.1 (VDD), SW73.1 (VDD), SW74.1 (VDD), SW75.1 (VDD), SW76.1 (VDD), SW77.1 (VDD), SW78.1 (VDD), SW79.1 (VDD), SW8.1 (VDD), SW80.1 (VDD), SW81.1 (VDD), SW82.1 (VDD), SW83.1 (VDD), SW84.1 (VDD), SW85.1 (VDD), SW86.1 (VDD), SW87.1 (VDD), SW88.1 (VDD), SW89.1 (VDD), SW9.1 (VDD), SW90.1 (VDD), SW91.1 (VDD), SW92.1 (VDD), SW93.1 (VDD), SW94.1 (VDD), SW95.1 (VDD), SW96.1 (VDD), SW97.1 (VDD), SW98.1 (VDD), SW99.1 (VDD)
- net +5VD: no longer C101.1, D1.2 (A2), J1.A9 (VBUS), J1.B9 (VBUS), SW103.2 (B)
- new net +5VP: C1.1, C10.1, C100.1, C101.1, C11.1, C12.1, C13.1, C14.1, C15.1, C16.1, C17.1, C18.1, C19.1, C2.1, C20.1, C21.1, C22.1, C23.1, C24.1, C25.1, C26.1, C27.1, C28.1, C29.1, C3.1, C30.1, C31.1, C32.1, C33.1, C34.1, C35.1, C36.1, C37.1, C38.1, C39.1, C4.1, C40.1, C41.1, C42.1, C43.1, C44.1, C45.1, C46.1, C47.1, C48.1, C49.1, C5.1, C50.1, C51.1, C52.1, C53.1, C54.1, C55.1, C56.1, C57.1, C58.1, C59.1, C6.1, C60.1, C61.1, C62.1, C63.1, C64.1, C65.1, C66.1, C67.1, C68.1, C69.1, C7.1, C70.1, C71.1, C72.1, C73.1, C74.1, C75.1, C76.1, C77.1, C78.1, C79.1, C8.1, C80.1, C81.1, C82.1, C83.1, C84.1, C85.1, C86.1, C87.1, C88.1, C89.1, C9.1, C90.1, C91.1, C92.1, C93.1, C94.1, C95.1, C96.1, C97.1, C98.1, C99.1, D1.2 (A2), J1.A9 (VBUS), J1.B9 (VBUS), SW1.1 (VDD), SW10.1 (VDD), SW100.1 (VDD), SW103.2 (B), SW104.2 (B), SW11.1 (VDD), SW12.1 (VDD), SW13.1 (VDD), SW14.1 (VDD), SW15.1 (VDD), SW16.1 (VDD), SW17.1 (VDD), SW18.1 (VDD), SW19.1 (VDD), SW2.1 (VDD), SW20.1 (VDD), SW21.1 (VDD), SW22.1 (VDD), SW23.1 (VDD), SW24.1 (VDD), SW25.1 (VDD), SW26.1 (VDD), SW27.1 (VDD), SW28.1 (VDD), SW29.1 (VDD), SW3.1 (VDD), SW30.1 (VDD), SW31.1 (VDD), SW32.1 (VDD), SW33.1 (VDD), SW34.1 (VDD), SW35.1 (VDD), SW36.1 (VDD), SW37.1 (VDD), SW38.1 (VDD), SW39.1 (VDD), SW4.1 (VDD), SW40.1 (VDD), SW41.1 (VDD), SW42.1 (VDD), SW43.1 (VDD), SW44.1 (VDD), SW45.1 (VDD), SW46.1 (VDD), SW47.1 (VDD), SW48.1 (VDD), SW49.1 (VDD), SW5.1 (VDD), SW50.1 (VDD), SW51.1 (VDD), SW52.1 (VDD), SW53.1 (VDD), SW54.1 (VDD), SW55.1 (VDD), SW56.1 (VDD), SW57.1 (VDD), SW58.1 (VDD), SW59.1 (VDD), SW6.1 (VDD), SW60.1 (VDD), SW61.1 (VDD), SW62.1 (VDD), SW63.1 (VDD), SW64.1 (VDD), SW65.1 (VDD), SW66.1 (VDD), SW67.1 (VDD), SW68.1 (VDD), SW69.1 (VDD), SW7.1 (VDD), SW70.1 (VDD), SW71.1 (VDD), SW72.1 (VDD), SW73.1 (VDD), SW74.1 (VDD), SW75.1 (VDD), SW76.1 (VDD), SW77.1 (VDD), SW78.1 (VDD), SW79.1 (VDD), SW8.1 (VDD), SW80.1 (VDD), SW81.1 (VDD), SW82.1 (VDD), SW83.1 (VDD), SW84.1 (VDD), SW85.1 (VDD), SW86.1 (VDD), SW87.1 (VDD), SW88.1 (VDD), SW89.1 (VDD), SW9.1 (VDD), SW90.1 (VDD), SW91.1 (VDD), SW92.1 (VDD), SW93.1 (VDD), SW94.1 (VDD), SW95.1 (VDD), SW96.1 (VDD), SW97.1 (VDD), SW98.1 (VDD), SW99.1 (VDD)

Commit message: Almost done, schematic
Parts:
- removed R2: 4.7 K, Resistor_SMD:R_1206_3216Metric, symbol Device:R
- added R43, R44, R45, R46, R47, R48, R49, R50, R51, R52, R53, R54, R55, R56, R57, R58, R59, R60, R61, R62: 220, symbol Device:R
Connections:
- net +5VD is gone; now on net +5VP: J2.1 (Pin_1)
- net spi_clk is gone; now on net spi_clk_lcd: LCD1.3 (SCK)
- net spi_data is gone; now on net spi_data_lcd: LCD1.4 (SDA)
- net audio_bclk: now also U1.22 (PA5); no longer U1.40 (PD8)
- net audio_din: now also U1.19 (PA2); no longer U1.44 (PA12)
- net audio_lrclk: now also U1.21 (PA4); no longer U1.47 (PA15)
- net audio_mode: now also U1.23 (PA6); no longer U1.43 (PA11)
- net col_1: now also R44.1
- net col_10: now also R55.2
- net col_2: now also R43.1
- net col_3: now also R45.1
- net col_4: now also R46.1
- net col_5: now also R47.1
- net col_6: now also R48.1
- net col_7: now also R49.1
- net col_8: now also R57.1
- net col_9: now also R56.1
- net dc_lcd: now also U1.59 (PB5)
- net esp_uart_rx: now also U1.17 (PA0); no longer U1.37 (PA9)
- net esp_uart_tx: now also U1.18 (PA1); no longer U1.42 (PA10)
- net key_1: now also U1.1 (PC11)
- net key_2: now also U1.2 (PC12)
- net reset_lcd: now also U1.58 (PB4)
- net rgb_data_3V: now also U1.64 (PC10)
- net row_1: now also R58.2
- net row_10: now also R52.2
- net row_2: now also R51.1
- net row_3: now also R50.1
- net row_4: now also R60.1
- net row_5: now also R61.1
- net row_6: now also R59.2
- net row_7: now also R62.2
- net row_8: now also R54.2
- net row_9: now also R53.2
- net spi_mem_clk: now also U1.30 (PB10); no longer U1.33 (PB13)
- net spi_mem_cs: now also U1.32 (PB12); no longer U1.36 (PA8)
- net spi_mem_miso: now also U1.29 (PB2); no longer U1.34 (PB14)
- net spi_mem_mosi: now also U1.31 (PB11); no longer U1.35 (PB15)
- net swclk: no longer U1.46 (PA14)
- net swdio: no longer U1.45 (PA13)
- net esp_reset: now reaches U1.16 (PC3)
- net esp_reset: now also U6.1 (~{RST})
- net at U1.37 (PA9): now also R59.1
- net at U1.38 (PC6): now also R61.2
- net at U1.39 (PC7): now also R60.2
- net at U1.41 (PD9): now also R51.2
- net at U1.42 (PA10): now also R58.1
- net at U1.48 (PC8): now also R56.2
- net at U1.49 (PC9): now also R57.2
- net at U1.50 (PD0): now also R49.2
- net at U1.51 (PD1): now also R48.2
- net at U1.52 (PD2): now also R47.2
- net at U1.53 (PD3): now also R46.2
- net at U1.54 (PD4): now also R45.2
- net at U1.55 (PD5): now also R43.2
- net at U1.56 (PD6): now also R44.2
- net spi_clk_lcd: now reaches U1.57 (PB3)
- net spi_data_lcd: now reaches U1.60 (PB6)
- net blk_lcd: now reaches U1.62 (PB8)
- net blk_lcd: now also LCD1.7 (BLK)
- new net: R52.1, U1.33 (PB13)
- new net: R53.1, U1.34 (PB14)
- new net: R54.1, U1.35 (PB15)
- new net: R62.1, U1.36 (PA8)
- new net: R50.2, U1.40 (PD8)
- new net: R55.1, U1.47 (PA15)
- no-connect marks 9 -> 37
Other:
- moved on the sheet: R22, R23, R24

Commit message: Schematic V2.0
Parts:
- removed C105, C106: 100n, Capacitor_SMD:C_1206_3216Metric, symbol Device:C
- removed R11, R5, R6: 1k, Resistor_SMD:R_1206_3216Metric, symbol Device:R
- removed R12, R13, R14: 10k, Resistor_SMD:R_1206_3216Metric, symbol Device:R
- removed SW101, SW102: SW_Push, Button_Switch_THT:SW_PUSH_6mm, symbol Switch:SW_Push
- added C113, C114: 100n, Capacitor_SMD:C_0805_2012Metric, symbol Device:C
- added R39, R40, R41: 10k, Resistor_SMD:R_0805_2012Metric, symbol Device:R
- added R42, R43, R44: 1k, Resistor_SMD:R_0805_2012Metric, symbol Device:R
- added SW103, SW104: SW_Push, Button_Switch_THT:SW_PUSH_6mm, symbol Switch:SW_Push
- C1, C10, C11, C12, C13, C14, C15, C16, C17, C18, C19, C2, C20, C25, C3, C4, C5, C55, C6, C7, C8, C9: footprint (none) -> Capacitor_SMD:C_0805_2012Metric
- C100: renamed from C95; footprint (none) -> Capacitor_SMD:C_0805_2012Metric
- C101: renamed from C97; footprint (none) -> Capacitor_SMD:C_0805_2012Metric
- C102: renamed from C99; footprint (none) -> Capacitor_SMD:C_0805_2012Metric
- C103: renamed from C82; footprint (none) -> Capacitor_SMD:C_0805_2012Metric
- C104: renamed from C84; footprint (none) -> Capacitor_SMD:C_0805_2012Metric
- C105: renamed from C86; footprint (none) -> Capacitor_SMD:C_0805_2012Metric
- C106: renamed from C88; footprint (none) -> Capacitor_SMD:C_0805_2012Metric
- C107: renamed from C90; footprint (none) -> Capacitor_SMD:C_0805_2012Metric
- C108: renamed from C92; footprint (none) -> Capacitor_SMD:C_0805_2012Metric
- C109: renamed from C94; footprint (none) -> Capacitor_SMD:C_0805_2012Metric
- C110: renamed from C96; footprint (none) -> Capacitor_SMD:C_0805_2012Metric
- C111: renamed from C98; footprint (none) -> Capacitor_SMD:C_0805_2012Metric
- C112: renamed from C100; footprint (none) -> Capacitor_SMD:C_0805_2012Metric
- C115: footprint Capacitor_SMD:C_1206_3216Metric -> Capacitor_SMD:C_0805_2012Metric
- C21: renamed from C104; footprint (none) -> Capacitor_SMD:C_0805_2012Metric
- C22: renamed from C101; footprint Capacitor_SMD:C_1206_3216Metric -> Capacitor_SMD:C_0805_2012Metric
- C23: renamed from C21; footprint (none) -> Capacitor_SMD:C_0805_2012Metric
- C24: renamed from C23; footprint (none) -> Capacitor_SMD:C_0805_2012Metric
- C26: renamed from C27; footprint (none) -> Capacitor_SMD:C_0805_2012Metric
- C27: renamed from C29; footprint (none) -> Capacitor_SMD:C_0805_2012Metric
- C28: renamed from C31; footprint (none) -> Capacitor_SMD:C_0805_2012Metric
- C29: renamed from C33; footprint (none) -> Capacitor_SMD:C_0805_2012Metric
- C30: renamed from C35; footprint (none) -> Capacitor_SMD:C_0805_2012Metric
- C31: renamed from C37; footprint (none) -> Capacitor_SMD:C_0805_2012Metric
- C32: renamed from C39; footprint (none) -> Capacitor_SMD:C_0805_2012Metric
- C33: renamed from C103; footprint (none) -> Capacitor_SMD:C_0805_2012Metric
- C34: renamed from C22; footprint (none) -> Capacitor_SMD:C_0805_2012Metric
- C35: renamed from C24; footprint (none) -> Capacitor_SMD:C_0805_2012Metric
- C36: renamed from C26; footprint (none) -> Capacitor_SMD:C_0805_2012Metric
- C37: renamed from C28; footprint (none) -> Capacitor_SMD:C_0805_2012Metric
- C38: renamed from C30; footprint (none) -> Capacitor_SMD:C_0805_2012Metric
- C39: renamed from C32; footprint (none) -> Capacitor_SMD:C_0805_2012Metric
- C40: renamed from C34; footprint (none) -> Capacitor_SMD:C_0805_2012Metric
- C41: renamed from C36; footprint (none) -> Capacitor_SMD:C_0805_2012Metric
- C42: renamed from C38; footprint (none) -> Capacitor_SMD:C_0805_2012Metric
- C43: renamed from C40; footprint (none) -> Capacitor_SMD:C_0805_2012Metric
- C44: renamed from C114; footprint (none) -> Capacitor_SMD:C_0805_2012Metric
- C45: renamed from C111; footprint (none) -> Capacitor_SMD:C_0805_2012Metric
- C46: renamed from C110; footprint (none) -> Capacitor_SMD:C_0805_2012Metric
- C47: renamed from C109; footprint (none) -> Capacitor_SMD:C_0805_2012Metric
- C48: renamed from C41; footprint (none) -> Capacitor_SMD:C_0805_2012Metric
- C49: renamed from C43; footprint (none) -> Capacitor_SMD:C_0805_2012Metric
- C50: renamed from C45; footprint (none) -> Capacitor_SMD:C_0805_2012Metric
- C51: renamed from C47; footprint (none) -> Capacitor_SMD:C_0805_2012Metric
- C52: renamed from C49; footprint (none) -> Capacitor_SMD:C_0805_2012Metric
- C53: renamed from C51; footprint (none) -> Capacitor_SMD:C_0805_2012Metric
- C54: renamed from C53; footprint (none) -> Capacitor_SMD:C_0805_2012Metric
- C56: renamed from C57; footprint (none) -> Capacitor_SMD:C_0805_2012Metric
- C57: renamed from C59; footprint (none) -> Capacitor_SMD:C_0805_2012Metric
- C58: renamed from C108; footprint (none) -> Capacitor_SMD:C_0805_2012Metric
- C59: renamed from C107; footprint (none) -> Capacitor_SMD:C_0805_2012Metric
- C60: renamed from C42; footprint (none) -> Capacitor_SMD:C_0805_2012Metric
- C61: renamed from C44; footprint (none) -> Capacitor_SMD:C_0805_2012Metric
- C62: renamed from C46; footprint (none) -> Capacitor_SMD:C_0805_2012Metric
- C63: renamed from C48; footprint (none) -> Capacitor_SMD:C_0805_2012Metric
- C64: renamed from C50; footprint (none) -> Capacitor_SMD:C_0805_2012Metric
- C65: renamed from C52; footprint (none) -> Capacitor_SMD:C_0805_2012Metric
- C66: renamed from C54; footprint (none) -> Capacitor_SMD:C_0805_2012Metric
- C67: renamed from C56; footprint (none) -> Capacitor_SMD:C_0805_2012Metric
- C68: renamed from C58; footprint (none) -> Capacitor_SMD:C_0805_2012Metric
- C69: renamed from C60; footprint (none) -> Capacitor_SMD:C_0805_2012Metric
- C70: renamed from C102; footprint Capacitor_SMD:C_1206_3216Metric -> Capacitor_SMD:C_0805_2012Metric
- C71: renamed from C61; footprint (none) -> Capacitor_SMD:C_0805_2012Metric
- C72: renamed from C63; footprint (none) -> Capacitor_SMD:C_0805_2012Metric
- C73: renamed from C65; footprint (none) -> Capacitor_SMD:C_0805_2012Metric
- C74: renamed from C67; footprint (none) -> Capacitor_SMD:C_0805_2012Metric
- C75: renamed from C69; footprint (none) -> Capacitor_SMD:C_0805_2012Metric
- C76: renamed from C71; footprint (none) -> Capacitor_SMD:C_0805_2012Metric
- C77: renamed from C73; footprint (none) -> Capacitor_SMD:C_0805_2012Metric
- C78: renamed from C75; footprint (none) -> Capacitor_SMD:C_0805_2012Metric
- C79: renamed from C77; footprint (none) -> Capacitor_SMD:C_0805_2012Metric
- C80: renamed from C79; footprint (none) -> Capacitor_SMD:C_0805_2012Metric
- C81: renamed from C113; footprint (none) -> Capacitor_SMD:C_0805_2012Metric
- C82: renamed from C112; footprint (none) -> Capacitor_SMD:C_0805_2012Metric
- C83: renamed from C62; footprint (none) -> Capacitor_SMD:C_0805_2012Metric
- C84: renamed from C64; footprint (none) -> Capacitor_SMD:C_0805_2012Metric
- C85: renamed from C66; footprint (none) -> Capacitor_SMD:C_0805_2012Metric
- C86: renamed from C68; footprint (none) -> Capacitor_SMD:C_0805_2012Metric
- C87: renamed from C70; footprint (none) -> Capacitor_SMD:C_0805_2012Metric
- C88: renamed from C72; footprint (none) -> Capacitor_SMD:C_0805_2012Metric
- C89: renamed from C74; footprint (none) -> Capacitor_SMD:C_0805_2012Metric
- C90: renamed from C76; footprint (none) -> Capacitor_SMD:C_0805_2012Metric
- C91: renamed from C78; footprint (none) -> Capacitor_SMD:C_0805_2012Metric
- C92: renamed from C80; footprint (none) -> Capacitor_SMD:C_0805_2012Metric
- C93: renamed from C81; footprint (none) -> Capacitor_SMD:C_0805_2012Metric
- C94: renamed from C83; footprint (none) -> Capacitor_SMD:C_0805_2012Metric
- C95: renamed from C85; footprint (none) -> Capacitor_SMD:C_0805_2012Metric
- C96: renamed from C87; footprint (none) -> Capacitor_SMD:C_0805_2012Metric
- C97: renamed from C89; footprint (none) -> Capacitor_SMD:C_0805_2012Metric
- C98: renamed from C91; footprint (none) -> Capacitor_SMD:C_0805_2012Metric
- C99: renamed from C93; footprint (none) -> Capacitor_SMD:C_0805_2012Metric
- LS1: footprint (none) -> Connector_PinHeader_2.54mm:PinHeader_1x02_P2.54mm_Vertical
- R1: footprint (none) -> Resistor_SMD:R_0805_2012Metric
- R10: renamed from R16; footprint (none) -> Resistor_SMD:R_0805_2012Metric
- R11: renamed from R10; footprint (none) -> Resistor_SMD:R_0805_2012Metric
- R12: renamed from R9; footprint (none) -> Resistor_SMD:R_0805_2012Metric
- R13: renamed from R3; footprint Resistor_SMD:R_1206_3216Metric -> Resistor_SMD:R_0805_2012Metric
- renumbered D2 to D1, D6 to D10, D92 to D100, D12 to D11, D21 to D12, D30 to D13, D39 to D14, D48 to D15, D57 to D16, D66 to D17, D75 to D18, D84 to D19, D3 to D2, D93 to D20, D1 to D21, D13 to D22, D22 to D23, D31 to D24, D40 to D25, D49 to D26, D58 to D27, D67 to D28, D76 to D29, D4 to D3, D85 to D30, D94 to D31, D14 to D32, D23 to D33, D32 to D34, D41 to D35, D50 to D36, D59 to D37, D68 to D38, D77 to D39, D5 to D4, D86 to D40, D95 to D41, D15 to D42, D24 to D43, D33 to D44, D42 to D45, D51 to D46, D60 to D47, D69 to D48, D78 to D49, D7 to D5, D87 to D50, D96 to D51, D16 to D52, D25 to D53, D34 to D54, D43 to D55, D52 to D56, D61 to D57, D70 to D58, D79 to D59, D8 to D6, D88 to D60, D97 to D61, D17 to D62, D26 to D63, D35 to D64, D44 to D65, D53 to D66, D62 to D67, D71 to D68, D80 to D69, D9 to D7, D89 to D70, D98 to D71, D18 to D72, D27 to D73, D36 to D74, D45 to D75, D54 to D76, D63 to D77, D72 to D78, D81 to D79, D10 to D8, D90 to D80, D99 to D81, D19 to D82, D28 to D83, D37 to D84, D46 to D85, D55 to D86, D64 to D87, D73 to D88, D82 to D89, D11 to D9, D91 to D90, D100 to D91, D20 to D92, D29 to D93, D38 to D94, D47 to D95, D56 to D96, D65 to D97, D74 to D98, D83 to D99, SW96 to SW100, SW98 to SW101, SW100 to SW102, SW103 to SW21, SW21 to SW22, SW25 to SW24, SW27 to SW25, SW29 to SW26, SW31 to SW27, SW33 to SW28, SW35 to SW29, SW37 to SW30, SW39 to SW31, SW22 to SW32, SW24 to SW33, SW26 to SW34, SW28 to SW35, SW30 to SW36, SW32 to SW37, SW34 to SW38, SW36 to SW39, SW38 to SW40, SW40 to SW41, SW41 to SW42, SW45 to SW44, SW47 to SW45, SW49 to SW46, SW51 to SW47, SW53 to SW48, SW55 to SW49, SW57 to SW50, SW59 to SW51, SW42 to SW52, SW44 to SW53, SW46 to SW54, SW48 to SW55, SW50 to SW56, SW52 to SW57, SW54 to SW58, SW56 to SW59, SW58 to SW60, SW60 to SW61, SW61 to SW62, SW65 to SW64, SW67 to SW65, SW69 to SW66, SW71 to SW67, SW73 to SW68, SW75 to SW69, SW77 to SW70, SW79 to SW71, SW62 to SW72, SW64 to SW73, SW66 to SW74, SW68 to SW75, SW70 to SW76, SW72 to SW77, SW74 to SW78, SW76 to SW79, SW78 to SW80, SW80 to SW81, SW81 to SW82, SW85 to SW84, SW87 to SW85, SW89 to SW86, SW91 to SW87, SW93 to SW88, SW95 to SW89, SW97 to SW90, SW99 to SW91, SW104 to SW92, SW82 to SW93, SW84 to SW94, SW86 to SW95, SW88 to SW96, SW90 to SW97, SW92 to SW98, SW94 to SW99, U3 to U1, U4 to U2, U2 to U3, U1 to U4
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Connections:
- net +3V3: now also R39.2, R40.2, R41.2
- net GND: now also C113.2, C114.2, SW103.1, SW104.1
- net key_1: now also C113.1, R40.1, R42.2
- net key_2: now also C114.1, R41.1, R43.2
- net stm32_reset: now also R39.1, R44.2
- net at SW105.2: now also R44.1
- net at U4.37 (PA9): now also R35.1
- net at U4.42 (PA10): now also R37.1
- new net: R43.1, SW104.2
- new net: R42.1, SW103.2
