File: schema_2/schema_2.kicad_sch (KiCad schematic)
At the start: 377 parts, among them J1 USB_C_Receptacle_PowerOnly_6P, J2 Conn_01x03_Pin, J3 Conn_01x04_Pin, SW103 SW_Push, SW104 SW_Push, SW105 SW_Push, SW21 SK12D07VG3, SW92 SK12D07VG3, U1 AP2112K-3.3, U2 W25Q128JVS, U3 74AHCT125, U4 STM32G070RBTx, U5 MAX98357A, U6 WEMOS_D1_mini, Y1 SX3M8.000M20F30TNN

Commit message: pcb start
Parts:
- D21: footprint Diode_SMD:D_SOD-882 -> Diode_SMD:D_SOD-882D
Connections:
- net col_2: now also D12.1 (K), D23.1 (K), D33.1 (K), D43.1 (K), D53.1 (K), D63.1 (K), D73.1 (K), D83.1 (K), D93.1 (K)
- net swclk: now also U4.46 (PA14)
- net swdio: now also U4.45 (PA13)
- net at U4.37 (PA9): now also R35.1
- net at U4.42 (PA10): now also R37.1
- no-connect marks 37 -> 36
Other:
- moved on the sheet: C1
Changed lines of the file:
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@@
 	)
 	(no_connect
-		(at 561.34 276.86)
-	)
-	(no_connect
 		(at 525.78 302.26)
 	)
@@
 	)
 	(no_connect
-		(at 561.34 274.32)
-	)
-	(no_connect
 		(at 525.78 292.1)
 	)
@@
 	)
 	(no_connect
+		(at 561.34 264.16)
+	)
+	(no_connect
 		(at 502.92 433.07)
 	)
@@
 	(wire
 		(pts
+			(xy 561.34 276.86) (xy 568.96 276.86)
+		)
+		(stroke
+			(width 0)
+			(type default)
+		)
+	)
+	(wire
+		(pts
 			(xy 228.6 240.03) (xy 232.41 240.03)
 		)
@@
 	(wire
 		(pts
+			(xy 85.09 140.97) (xy 85.09 143.51)
+		)
+		(stroke
+			(width 0)
+			(type default)
+		)
+	)
+	(wire
+		(pts
 			(xy 137.16 407.67) (xy 140.97 407.67)
 		)
@@
 	(wire
 		(pts
+			(xy 561.34 274.32) (xy 568.96 274.32)
+		)
+		(stroke
+			(width 0)
+			(type default)
+		)
+	)
+	(wire
+		(pts
 			(xy 495.3 279.4) (xy 518.16 279.4)
 		)
@@
 	(wire
 		(pts
+			(xy 85.09 392.43) (xy 85.09 394.97)
+		)
+		(stroke
+			(width 0)
+			(type default)
+		)
+	)
+	(wire
+		(pts
 			(xy 106.68 30.48) (xy 106.68 34.29)
 		)
@@
 	(wire
 		(pts
+			(xy 85.09 434.34) (xy 85.09 436.88)
+		)
+		(stroke
+			(width 0)
+			(type default)
+		)
+	)
+	(wire
+		(pts
 			(xy 54.61 101.6) (xy 54.61 99.06)
 		)
@@
 	(wire
 		(pts
+			(xy 85.09 224.79) (xy 85.09 227.33)
+		)
+		(stroke
+			(width 0)
+			(type default)
+		)
+	)
+	(wire
+		(pts
 			(xy 146.05 269.24) (xy 146.05 266.7)
 		)
@@
 	(wire
 		(pts
+			(xy 85.09 99.06) (xy 85.09 101.6)
+		)
+		(stroke
+			(width 0)
+			(type default)
+		)
+	)
+	(wire
+		(pts
 			(xy 495.3 307.34) (xy 502.92 307.34)
 		)
@@
 	(wire
 		(pts
-			(xy 57.15 30.48) (xy 55.88 30.48)
-		)
-		(stroke
-			(width 0)
-			(type default)
-		)
-	)
-	(wire
-		(pts
 			(xy 207.01 59.69) (xy 207.01 57.15)
 		)
@@
 	(wire
 		(pts
+			(xy 85.09 308.61) (xy 85.09 311.15)
+		)
+		(stroke
+			(width 0)
+			(type default)
+		)
+	)
+	(wire
+		(pts
 			(xy 176.53 101.3012) (xy 176.53 99.06)
 		)
@@
 	(wire
 		(pts
+			(xy 55.88 30.48) (xy 58.42 30.48)
+		)
+		(stroke
+			(width 0)
+			(type default)
+		)
+	)
+	(wire
+		(pts
 			(xy 198.12 196.85) (xy 198.12 198.12)
 		)
@@
 	(wire
 		(pts
-			(xy 45.72 30.48) (xy 49.53 30.48)
+			(xy 45.72 30.48) (xy 48.26 30.48)
 		)
 		(stroke
@@
 	(wire
 		(pts
+			(xy 85.09 350.52) (xy 85.09 353.06)
+		)
+		(stroke
+			(width 0)
+			(type default)
+		)
+	)
+	(wire
+		(pts
 			(xy 76.2 238.76) (xy 76.2 240.03)
 		)
@@
 	(wire
 		(pts
+			(xy 85.09 266.7) (xy 85.09 269.24)
+		)
+		(stroke
+			(width 0)
+			(type default)
+		)
+	)
+	(wire
+		(pts
 			(xy 298.45 293.37) (xy 311.15 293.37)
 		)
@@
 	(wire
 		(pts
-			(xy 267.97 353.06) (xy 267.97 350.52)
+			(xy 85.09 182.88) (xy 85.09 185.42)
 		)
 		(stroke
@@
 	(wire
 		(pts
-			(xy 331.47 30.48) (xy 330.2 30.48)
+			(xy 267.97 353.06) (xy 267.97 350.52)
 		)
 		(stroke
@@
 	(wire
 		(pts
-			(xy 495.3 274.32) (xy 502.92 274.32)
+			(xy 331.47 30.48) (xy 330.2 30.48)
 		)
 		(stroke
@@
 	(wire
 		(pts
-			(xy 198.12 364.49) (xy 198.12 365.76)
+			(xy 495.3 274.32) (xy 502.92 274.32)
 		)
 		(stroke
@@
 	(wire
 		(pts
-			(xy 259.08 30.48) (xy 259.08 34.29)
+			(xy 198.12 364.49) (xy 198.12 365.76)
 		)
 		(stroke
@@
 	(wire
 		(pts
-			(xy 176.53 49.8288) (xy 176.53 49.53)
+			(xy 259.08 30.48) (xy 259.08 34.29)
 		)
 		(stroke
@@
 	(wire
 		(pts
-			(xy 176.53 59.69) (xy 176.53 57.4488)
+			(xy 176.53 59.69) (xy 176.53 57.15)
 		)
 		(stroke
@@
 		)
 	)
+	(label "swclk"
+		(at 568.96 276.86 0)
+		(effects
+			(font
+				(size 1.27 1.27)
+			)
+			(justify left bottom)
+		)
+	)
 	(label "key_1"
 		(at 156.21 494.03 0)
@@
 		)
 	)
+	(label "swdio"
+		(at 568.96 274.32 0)
+		(effects
+			(font
+				(size 1.27 1.27)
+			)
+			(justify left bottom)
+		)
+	)
 	(label "col_10"
 		(at 328.93 311.15 0)
@@
 	(symbol
 		(lib_id "power:GND")
-		(at 55.88 30.48 90)
+		(at 58.42 30.48 90)
 		(unit 1)
 		(body_style 1)
@@
 		(fields_autoplaced yes)
 		(property "Reference" "#PWR011"
-			(at 62.23 30.48 0)
+			(at 64.77 30.48 0)
 			(hide yes)
 			(show_name no)
@@
 		)
 		(property "Value" "GND"
-			(at 59.69 30.4799 90)
+			(at 62.23 30.4799 90)
 			(show_name no)
 			(do_not_autoplace no)
@@
 		)
 		(property "Footprint" ""
-			(at 55.88 30.48 0)
+			(at 58.42 30.48 0)
 			(hide yes)
 			(show_name no)
@@
 		)
 		(property "Datasheet" ""
-			(at 55.88 30.48 0)
+			(at 58.42 30.48 0)
 			(hide yes)
 			(show_name no)
@@
 		)
 		(property "Description" "Power symbol creates a global label with name \"GND\" , ground"
-			(at 55.88 30.48 0)
+			(at 58.42 30.48 0)
 			(hide yes)
 			(show_name no)
@@
 	(symbol
 		(lib_id "Device:C")
-		(at 53.34 30.48 90)
+		(at 52.07 30.48 90)
 		(unit 1)
 		(body_style 1)
@@
 		(fields_autoplaced yes)
 		(property "Reference" "C1"
-			(at 53.34 22.86 90)
+			(at 52.07 22.86 90)
 			(show_name no)
 			(do_not_autoplace no)
@@
 		)
 		(property "Value" "100n"
-			(at 53.34 25.4 90)
+			(at 52.07 25.4 90)
 			(show_name no)
 			(do_not_autoplace no)
@@
 		)
 		(property "Footprint" "Capacitor_SMD:C_0805_2012Metric"
-			(at 57.15 29.5148 0)
+			(at 55.88 29.5148 0)
 			(hide yes)
 			(show_name no)
@@
 		)
 		(property "Datasheet" ""
-			(at 53.34 30.48 0)
+			(at 52.07 30.48 0)
 			(hide yes)
 			(show_name no)
@@
 		)
 		(property "Description" "Unpolarized capacitor"
-			(at 53.34 30.48 0)
+			(at 52.07 30.48 0)
 			(hide yes)
 			(show_name no)
@@
 	(symbol
 		(lib_id "Device:D")
-		(at 176.53 53.6388 90)
+		(at 176.53 53.34 90)
 		(unit 1)
 		(body_style 1)
@@
 		(fields_autoplaced yes)
 		(property "Reference" "D10"
-			(at 179.07 52.3687 90)
+			(at 179.07 52.0699 90)
 			(show_name no)
 			(do_not_autoplace no)
@@
 		)
 		(property "Value" "SM4007PL"
-			(at 179.07 54.9087 90)
+			(at 179.07 54.6099 90)
 			(show_name no)
 			(do_not_autoplace no)
@@
 		)
 		(property "Footprint" "Diode_SMD:D_SOD-123F"
-			(at 176.53 53.6388 0)
+			(at 176.53 53.34 0)
 			(hide yes)
 			(show_name no)
@@
 		)
 		(property "Datasheet" ""
-			(at 176.53 53.6388 0)
+			(at 176.53 53.34 0)
 			(hide yes)
 			(show_name no)
@@
 		)
 		(property "Description" "Diode"
-			(at 176.53 53.6388 0)
+			(at 176.53 53.34 0)
 			(hide yes)
 			(show_name no)
@@
 		)
 		(property "Sim.Device" "D"
-			(at 176.53 53.6388 0)
+			(at 176.53 53.34 0)
 			(hide yes)
 			(show_name no)
@@
 		)
 		(property "Sim.Pins" "1=K 2=A"
-			(at 176.53 53.6388 0)
+			(at 176.53 53.34 0)
 			(hide yes)
 			(show_name no)
@@
 			)
 		)
-		(property "Footprint" "Diode_SMD:D_SOD-882"
+		(property "Footprint" "Diode_SMD:D_SOD-882D"
 			(at 449.58 113.03 0)
 			(hide yes)

Commit message: 30.10.2026 (1)
Parts:
- renumbered D9 to D10, D10 to D5, D5 to D6, D6 to D7, D7 to D8, D8 to D9
Connections:
- net at U4.37 (PA9): now also R35.1
- net at U4.42 (PA10): now also R37.1
Changed lines of the file:
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@@
 		(dnp no)
 		(fields_autoplaced yes)
-		(property "Reference" "D5"
+		(property "Reference" "D6"
 			(at 209.55 52.0699 90)
 			(show_name no)
@@
 			(project "schema_2"
 				(path "/684f36b5-8ccc-4bbc-873e-3d1c5cfac569"
-					(reference "D5")
+					(reference "D6")
 					(unit 1)
 				)
@@
 		(dnp no)
 		(fields_autoplaced yes)
-		(property "Reference" "D9"
+		(property "Reference" "D10"
 			(at 331.47 52.0699 90)
 			(show_name no)
@@
 			(project "schema_2"
 				(path "/684f36b5-8ccc-4bbc-873e-3d1c5cfac569"
-					(reference "D9")
+					(reference "D10")
 					(unit 1)
 				)
@@
 		(dnp no)
 		(fields_autoplaced yes)
-		(property "Reference" "D6"
+		(property "Reference" "D7"
 			(at 240.03 52.0699 90)
 			(show_name no)
@@
 			(project "schema_2"
 				(path "/684f36b5-8ccc-4bbc-873e-3d1c5cfac569"
-					(reference "D6")
+					(reference "D7")
 					(unit 1)
 				)
@@
 		(dnp no)
 		(fields_autoplaced yes)
-		(property "Reference" "D10"
+		(property "Reference" "D5"
 			(at 179.07 52.0699 90)
 			(show_name no)
@@
 			(project "schema_2"
 				(path "/684f36b5-8ccc-4bbc-873e-3d1c5cfac569"
-					(reference "D10")
+					(reference "D5")
 					(unit 1)
 				)
@@
 		(dnp no)
 		(fields_autoplaced yes)
-		(property "Reference" "D7"
+		(property "Reference" "D8"
 			(at 270.51 52.0699 90)
 			(show_name no)
@@
 			(project "schema_2"
 				(path "/684f36b5-8ccc-4bbc-873e-3d1c5cfac569"
-					(reference "D7")
+					(reference "D8")
 					(unit 1)
 				)
@@
 		(dnp no)
 		(fields_autoplaced yes)
-		(property "Reference" "D8"
+		(property "Reference" "D9"
 			(at 300.99 52.0699 90)
 			(show_name no)
@@
 			(project "schema_2"
 				(path "/684f36b5-8ccc-4bbc-873e-3d1c5cfac569"
-					(reference "D8")
+					(reference "D9")
 					(unit 1)
 				)
