File: schema_2/schema_2.kicad_sch (KiCad schematic)
At the start: 377 parts, among them J1 USB_C_Receptacle_PowerOnly_6P, J2 Conn_01x03_Pin, J3 Conn_01x04_Pin, SW103 SW_Push, SW104 SW_Push, SW105 SW_Push, SW21 SK12D07VG3, SW92 SK12D07VG3, U1 AP2112K-3.3, U2 W25Q128JVS, U3 74AHCT125, U4 STM32G070RBTx, U5 MAX98357A, U6 WEMOS_D1_mini, Y1 SX3M8.000M20F30TNN

Commit message: 30.10.2026 (3)
Parts:
- R1: value R -> 1k
Connections:
- net +5V: no longer R13.1, R14.1, R15.1
- net +5VP: now also R13.1, R14.1, R15.1
- net at U4.37 (PA9): now also R35.1
- net at U4.42 (PA10): now also R37.1

Commit message: Connect all leds in snake style
Connections:
- net rgb_data_5V: now also SW10.4 (DIN); no longer SW1.4 (DIN)
- net led_56: now reaches SW57.2 (DOUT), SW58.4 (DIN)
- net led_55: now reaches SW56.2 (DOUT), SW57.4 (DIN)
- net led_54: now reaches SW55.2 (DOUT), SW56.4 (DIN)
- net led_62: now reaches SW69.4 (DIN)
- net led_62: now also SW70.2 (DOUT); no longer SW68.2 (DOUT)
- net led_63: now reaches SW68.4 (DIN)
- net led_63: now also SW69.2 (DOUT); no longer SW67.2 (DOUT)
- net led_19: now reaches SW19.2 (DOUT), SW20.4 (DIN)
- net led_18: now reaches SW18.2 (DOUT), SW19.4 (DIN)
- net led_17: now reaches SW17.2 (DOUT), SW18.4 (DIN)
- net at U4.37 (PA9): now also R35.1
- net at U4.42 (PA10): now also R37.1
- net led_40: now reaches SW51.4 (DIN)
- net led_40: now also SW41.2 (DOUT); no longer SW50.2 (DOUT)
- net led_41: now reaches SW50.4 (DIN)
- net led_41: now also SW51.2 (DOUT); no longer SW49.2 (DOUT)
- net led_52: now reaches SW53.2 (DOUT), SW54.4 (DIN)
- net led_51: now reaches SW52.2 (DOUT), SW53.4 (DIN)
- net led_26: now reaches SW25.4 (DIN)
- net led_26: now also SW26.2 (DOUT); no longer SW24.2 (DOUT)
- net led_27: now reaches SW24.4 (DIN)
- net led_27: now also SW25.2 (DOUT); no longer SW23.2 (DOUT)
- net led_57: now reaches SW58.2 (DOUT), SW59.4 (DIN)
- net led_99: now reaches SW101.2 (DOUT), SW102.4 (DIN)
- net led_98: now reaches SW100.2 (DOUT), SW101.4 (DIN)
- net led_1: now reaches SW9.4 (DIN)
- net led_1: now also SW10.2 (DOUT); no longer SW8.2 (DOUT)
- net led_2: now reaches SW8.4 (DIN)
- net led_2: now also SW9.2 (DOUT); no longer SW7.2 (DOUT)
- net led_92: now reaches SW94.2 (DOUT), SW95.4 (DIN)
- net led_91: now reaches SW93.2 (DOUT), SW94.4 (DIN)
- net led_44: now reaches SW47.4 (DIN)
- net led_44: now also SW48.2 (DOUT); no longer SW46.2 (DOUT)
- net led_45: now reaches SW46.4 (DIN)
- net led_45: now also SW47.2 (DOUT); no longer SW45.2 (DOUT)
- net led_38: now reaches SW39.2 (DOUT), SW40.4 (DIN)
- net led_37: now reaches SW38.2 (DOUT), SW39.4 (DIN)
- net led_82: now reaches SW89.4 (DIN)
- net led_82: now also SW90.2 (DOUT); no longer SW88.2 (DOUT)
- net led_83: now reaches SW88.4 (DIN)
- net led_83: now also SW89.2 (DOUT); no longer SW87.2 (DOUT)
- net led_3: now reaches SW7.4 (DIN)
- net led_3: now also SW8.2 (DOUT); no longer SW6.2 (DOUT)
- net led_81: now reaches SW90.4 (DIN)
- net led_81: now also SW91.2 (DOUT); no longer SW89.2 (DOUT)
- net led_86: now reaches SW85.4 (DIN)
- net led_86: now also SW86.2 (DOUT); no longer SW84.2 (DOUT)
- net led_87: now reaches SW84.4 (DIN)
- net led_87: now also SW85.2 (DOUT); no longer SW83.2 (DOUT)
- net led_39: now reaches SW40.2 (DOUT), SW41.4 (DIN)
- net led_22: now reaches SW29.4 (DIN)
- net led_22: now also SW30.2 (DOUT); no longer SW28.2 (DOUT)
- net led_23: now reaches SW28.4 (DIN)
- net led_23: now also SW29.2 (DOUT); no longer SW27.2 (DOUT)
- net led_77: now reaches SW78.2 (DOUT), SW79.4 (DIN)
- net led_76: now reaches SW77.2 (DOUT), SW78.4 (DIN)
- net led_28: now reaches SW23.4 (DIN)
- net led_28: now also SW24.2 (DOUT); no longer SW22.2 (DOUT)
- net led_6: now reaches SW4.4 (DIN)
- net led_6: now also SW5.2 (DOUT); no longer SW3.2 (DOUT)
- net led_7: now reaches SW3.4 (DIN)
- net led_7: now also SW4.2 (DOUT); no longer SW2.2 (DOUT)
- net led_94: now reaches SW96.2 (DOUT), SW97.4 (DIN)
- net led_93: now reaches SW95.2 (DOUT), SW96.4 (DIN)
- net led_67: now reaches SW64.4 (DIN)
- net led_67: now also SW65.2 (DOUT); no longer SW63.2 (DOUT)
- net led_68: now reaches SW63.4 (DIN)
- net led_68: now also SW64.2 (DOUT); no longer SW62.2 (DOUT)
- net led_12: now reaches SW12.2 (DOUT), SW13.4 (DIN)
- net led_11: now reaches SW11.2 (DOUT), SW12.4 (DIN)
- net led_53: now reaches SW54.2 (DOUT), SW55.4 (DIN)
- net led_34: now reaches SW35.2 (DOUT), SW36.4 (DIN)
- net led_33: now reaches SW34.2 (DOUT), SW35.4 (DIN)
- net led_20: now reaches SW31.4 (DIN)
- net led_20: now also SW20.2 (DOUT); no longer SW30.2 (DOUT)
- net led_21: now reaches SW30.4 (DIN)
- net led_21: now also SW31.2 (DOUT); no longer SW29.2 (DOUT)
- net led_13: now reaches SW13.2 (DOUT), SW14.4 (DIN)
- net led_95: now reaches SW97.2 (DOUT), SW98.4 (DIN)
- net led_59: now reaches SW60.2 (DOUT), SW61.4 (DIN)
- net led_47: now reaches SW44.4 (DIN)
- net led_47: now also SW45.2 (DOUT); no longer SW43.2 (DOUT)
- net led_48: now reaches SW43.4 (DIN)
- net led_48: now also SW44.2 (DOUT); no longer SW42.2 (DOUT)
- net led_46: now reaches SW45.4 (DIN)
- net led_46: now also SW46.2 (DOUT); no longer SW44.2 (DOUT)
- net led_4: now reaches SW6.4 (DIN)
- net led_4: now also SW7.2 (DOUT); no longer SW5.2 (DOUT)
- net led_5: now reaches SW5.4 (DIN)
- net led_5: now also SW6.2 (DOUT); no longer SW4.2 (DOUT)
- net led_75: now reaches SW76.2 (DOUT), SW77.4 (DIN)
- net led_74: now reaches SW75.2 (DOUT), SW76.4 (DIN)
- net led_16: now reaches SW16.2 (DOUT), SW17.4 (DIN)
- net led_15: now reaches SW15.2 (DOUT), SW16.4 (DIN)
- net led_36: now reaches SW37.2 (DOUT), SW38.4 (DIN)
- net led_31: now reaches SW32.2 (DOUT), SW33.4 (DIN)
- net led_32: now reaches SW33.2 (DOUT), SW34.4 (DIN)
- net led_79: now reaches SW80.2 (DOUT), SW81.4 (DIN)
- net led_78: now reaches SW79.2 (DOUT), SW80.4 (DIN)
- net led_24: now reaches SW27.4 (DIN)
- net led_24: now also SW28.2 (DOUT); no longer SW26.2 (DOUT)
- net led_25: now reaches SW26.4 (DIN)
- net led_25: now also SW27.2 (DOUT); no longer SW25.2 (DOUT)
- net led_72: now reaches SW73.2 (DOUT), SW74.4 (DIN)
- net led_71: now reaches SW72.2 (DOUT), SW73.4 (DIN)
- net led_60: now reaches SW71.4 (DIN)
- net led_60: now also SW61.2 (DOUT); no longer SW70.2 (DOUT)
- net led_61: now reaches SW70.4 (DIN)
- net led_61: now also SW71.2 (DOUT); no longer SW69.2 (DOUT)
- net led_73: now reaches SW74.2 (DOUT), SW75.4 (DIN)
- net led_14: now reaches SW14.2 (DOUT), SW15.4 (DIN)
- net led_58: now reaches SW59.2 (DOUT), SW60.4 (DIN)
- net led_80: now reaches SW91.4 (DIN)
- net led_80: now also SW81.2 (DOUT); no longer SW90.2 (DOUT)
- net led_42: now reaches SW49.4 (DIN)
- net led_42: now also SW50.2 (DOUT); no longer SW48.2 (DOUT)
- net led_10: now reaches SW1.2 (DOUT)
- net led_10: now also SW11.4 (DIN); no longer SW2.4 (DIN)
- net led_96: now reaches SW98.2 (DOUT), SW99.4 (DIN)
- net led_43: now reaches SW48.4 (DIN)
- net led_43: now also SW49.2 (DOUT); no longer SW47.2 (DOUT)
- net led_84: now reaches SW87.4 (DIN)
- net led_84: now also SW88.2 (DOUT); no longer SW86.2 (DOUT)
- net led_85: now reaches SW86.4 (DIN)
- net led_85: now also SW87.2 (DOUT); no longer SW85.2 (DOUT)
- net led_65: now reaches SW66.4 (DIN)
- net led_65: now also SW67.2 (DOUT); no longer SW65.2 (DOUT)
- net led_66: now reaches SW65.4 (DIN)
- net led_66: now also SW66.2 (DOUT); no longer SW64.2 (DOUT)
- net led_97: now reaches SW100.4 (DIN), SW99.2 (DOUT)
- net led_35: now reaches SW36.2 (DOUT), SW37.4 (DIN)
- net led_88: now reaches SW83.4 (DIN)
- net led_88: now also SW84.2 (DOUT); no longer SW82.2 (DOUT)
- net led_64: now reaches SW67.4 (DIN)
- net led_64: now also SW68.2 (DOUT); no longer SW66.2 (DOUT)
- removed net led_out_1: SW10.2 (DOUT), SW11.4 (DIN)
- net led_out_2 renamed led_29
- net led_29: now also SW23.2 (DOUT); no longer SW20.2 (DOUT)
- net led_out_3 renamed led_30
- net led_30: now also SW22.2 (DOUT); no longer SW31.2 (DOUT)
- net led_out_4 renamed led_49
- net led_49: now also SW43.2 (DOUT); no longer SW41.2 (DOUT)
- net led_out_5 renamed led_50
- net led_50: now also SW42.2 (DOUT); no longer SW51.2 (DOUT)
- net led_out_6 renamed led_69
- net led_69: now also SW63.2 (DOUT); no longer SW61.2 (DOUT)
- net led_out_7 renamed led_70
- net led_70: now also SW62.2 (DOUT); no longer SW71.2 (DOUT)
- net led_out_8 renamed led_89
- net led_89: now also SW83.2 (DOUT); no longer SW81.2 (DOUT)
- net led_out_9 renamed led_90
- net led_90: now also SW82.2 (DOUT); no longer SW91.2 (DOUT)
- new net led_8: SW2.4 (DIN), SW3.2 (DOUT)
- new net led_9: SW1.4 (DIN), SW2.2 (DOUT)
Other:
- note added: "switches: "snake" connection"

Commit message: Update schematic and pcb with new snake connection
Parts:
- SW1, SW10, SW2, SW22, SW23, SW24, SW25, SW26, SW27, SW28, SW29, SW3, SW30, SW31, SW4, SW42, SW43, SW44, SW45, SW46, SW47, SW48, SW49, SW5, SW50, SW51, SW6, SW62, SW63, SW64, SW65, SW66, SW67, SW68, SW69, SW7, SW70, SW71, SW8, SW82, SW83, SW84, SW85, SW86, SW87, SW88, SW89, SW9, SW90, SW91: footprint sw_led:SW_MX_1u_SK6812MINI-E_ROTATE -> sw_led:SW_MX_1u_SK6812MINI-E
Connections:
- net at U4.37 (PA9): now also R35.1
- net at U4.42 (PA10): now also R37.1
Changed lines of the file:
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@@
 			)
 		)
-		(property "Footprint" "sw_led:SW_MX_1u_SK6812MINI-E_ROTATE"
+		(property "Footprint" "sw_led:SW_MX_1u_SK6812MINI-E"
 			(at 228.6 287.02 0)
 			(hide yes)
@@
 			)
 		)
-		(property "Footprint" "sw_led:SW_MX_1u_SK6812MINI-E_ROTATE"
+		(property "Footprint" "sw_led:SW_MX_1u_SK6812MINI-E"
 			(at 289.56 203.2 0)
 			(hide yes)
@@
 			)
 		)
-		(property "Footprint" "sw_led:SW_MX_1u_SK6812MINI-E_ROTATE"
+		(property "Footprint" "sw_led:SW_MX_1u_SK6812MINI-E"
 			(at 106.68 119.38 0)
 			(hide yes)
@@
 			)
 		)
-		(property "Footprint" "sw_led:SW_MX_1u_SK6812MINI-E_ROTATE"
+		(property "Footprint" "sw_led:SW_MX_1u_SK6812MINI-E"
 			(at 259.08 35.56 0)
 			(hide yes)
@@
 			)
 		)
-		(property "Footprint" "sw_led:SW_MX_1u_SK6812MINI-E_ROTATE"
+		(property "Footprint" "sw_led:SW_MX_1u_SK6812MINI-E"
 			(at 167.64 203.2 0)
 			(hide yes)
@@
 			)
 		)
-		(property "Footprint" "sw_led:SW_MX_1u_SK6812MINI-E_ROTATE"
+		(property "Footprint" "sw_led:SW_MX_1u_SK6812MINI-E"
 			(at 228.6 370.84 0)
 			(hide yes)
@@
 			)
 		)
-		(property "Footprint" "sw_led:SW_MX_1u_SK6812MINI-E_ROTATE"
+		(property "Footprint" "sw_led:SW_MX_1u_SK6812MINI-E"
 			(at 228.6 35.56 0)
 			(hide yes)
@@
 			)
 		)
-		(property "Footprint" "sw_led:SW_MX_1u_SK6812MINI-E_ROTATE"
+		(property "Footprint" "sw_led:SW_MX_1u_SK6812MINI-E"
 			(at 259.08 370.84 0)
 			(hide yes)
@@
 			)
 		)
-		(property "Footprint" "sw_led:SW_MX_1u_SK6812MINI-E_ROTATE"
+		(property "Footprint" "sw_led:SW_MX_1u_SK6812MINI-E"
 			(at 106.68 370.84 0)
 			(hide yes)
@@
 			)
 		)
-		(property "Footprint" "sw_led:SW_MX_1u_SK6812MINI-E_ROTATE"
+		(property "Footprint" "sw_led:SW_MX_1u_SK6812MINI-E"
 			(at 228.6 119.38 0)
 			(hide yes)
@@
 			)
 		)
-		(property "Footprint" "sw_led:SW_MX_1u_SK6812MINI-E_ROTATE"
+		(property "Footprint" "sw_led:SW_MX_1u_SK6812MINI-E"
 			(at 289.56 35.56 0)
 			(hide yes)
@@
 			)
 		)
-		(property "Footprint" "sw_led:SW_MX_1u_SK6812MINI-E_ROTATE"
+		(property "Footprint" "sw_led:SW_MX_1u_SK6812MINI-E"
 			(at 45.72 119.38 0)
 			(hide yes)
@@
 			)
 		)
-		(property "Footprint" "sw_led:SW_MX_1u_SK6812MINI-E_ROTATE"
+		(property "Footprint" "sw_led:SW_MX_1u_SK6812MINI-E"
 			(at 106.68 35.56 0)
 			(hide yes)
@@
 			)
 		)
-		(property "Footprint" "sw_led:SW_MX_1u_SK6812MINI-E_ROTATE"
+		(property "Footprint" "sw_led:SW_MX_1u_SK6812MINI-E"
 			(at 76.2 287.02 0)
 			(hide yes)
@@
 			)
 		)
-		(property "Footprint" "sw_led:SW_MX_1u_SK6812MINI-E_ROTATE"
+		(property "Footprint" "sw_led:SW_MX_1u_SK6812MINI-E"
 			(at 320.04 35.56 0)
 			(hide yes)
@@
 			)
 		)
-		(property "Footprint" "sw_led:SW_MX_1u_SK6812MINI-E_ROTATE"
+		(property "Footprint" "sw_led:SW_MX_1u_SK6812MINI-E"
 			(at 289.56 119.38 0)
 			(hide yes)
@@
 			)
 		)
-		(property "Footprint" "sw_led:SW_MX_1u_SK6812MINI-E_ROTATE"
+		(property "Footprint" "sw_led:SW_MX_1u_SK6812MINI-E"
 			(at 76.2 203.2 0)
 			(hide yes)
@@
 			)
 		)
-		(property "Footprint" "sw_led:SW_MX_1u_SK6812MINI-E_ROTATE"
+		(property "Footprint" "sw_led:SW_MX_1u_SK6812MINI-E"
 			(at 137.16 203.2 0)
 			(hide yes)
@@
 			)
 		)
-		(property "Footprint" "sw_led:SW_MX_1u_SK6812MINI-E_ROTATE"
+		(property "Footprint" "sw_led:SW_MX_1u_SK6812MINI-E"
 			(at 167.64 35.56 0)
 			(hide yes)
@@
 			)
 		)
-		(property "Footprint" "sw_led:SW_MX_1u_SK6812MINI-E_ROTATE"
+		(property "Footprint" "sw_led:SW_MX_1u_SK6812MINI-E"
 			(at 45.72 203.2 0)
 			(hide yes)
@@
 			)
 		)
-		(property "Footprint" "sw_led:SW_MX_1u_SK6812MINI-E_ROTATE"
+		(property "Footprint" "sw_led:SW_MX_1u_SK6812MINI-E"
 			(at 259.08 119.38 0)
 			(hide yes)
@@
 			)
 		)
-		(property "Footprint" "sw_led:SW_MX_1u_SK6812MINI-E_ROTATE"
+		(property "Footprint" "sw_led:SW_MX_1u_SK6812MINI-E"
 			(at 198.12 35.56 0)
 			(hide yes)
@@
 			)
 		)
-		(property "Footprint" "sw_led:SW_MX_1u_SK6812MINI-E_ROTATE"
+		(property "Footprint" "sw_led:SW_MX_1u_SK6812MINI-E"
 			(at 167.64 119.38 0)
 			(hide yes)
@@
 			)
 		)
-		(property "Footprint" "sw_led:SW_MX_1u_SK6812MINI-E_ROTATE"
+		(property "Footprint" "sw_led:SW_MX_1u_SK6812MINI-E"
 			(at 289.56 287.02 0)
 			(hide yes)
@@
 			)
 		)
-		(property "Footprint" "sw_led:SW_MX_1u_SK6812MINI-E_ROTATE"
+		(property "Footprint" "sw_led:SW_MX_1u_SK6812MINI-E"
 			(at 45.72 287.02 0)
 			(hide yes)
@@
 			)
 		)
-		(property "Footprint" "sw_led:SW_MX_1u_SK6812MINI-E_ROTATE"
+		(property "Footprint" "sw_led:SW_MX_1u_SK6812MINI-E"
 			(at 198.12 119.38 0)
 			(hide yes)
@@
 			)
 		)
-		(property "Footprint" "sw_led:SW_MX_1u_SK6812MINI-E_ROTATE"
+		(property "Footprint" "sw_led:SW_MX_1u_SK6812MINI-E"
 			(at 320.04 370.84 0)
 			(hide yes)
@@
 			)
 		)
-		(property "Footprint" "sw_led:SW_MX_1u_SK6812MINI-E_ROTATE"
+		(property "Footprint" "sw_led:SW_MX_1u_SK6812MINI-E"
 			(at 259.08 203.2 0)
 			(hide yes)
@@
 			)
 		)
-		(property "Footprint" "sw_led:SW_MX_1u_SK6812MINI-E_ROTATE"
+		(property "Footprint" "sw_led:SW_MX_1u_SK6812MINI-E"
 			(at 45.72 35.56 0)
 			(hide yes)
@@
 			)
 		)
-		(property "Footprint" "sw_led:SW_MX_1u_SK6812MINI-E_ROTATE"
+		(property "Footprint" "sw_led:SW_MX_1u_SK6812MINI-E"
 			(at 137.16 119.38 0)
 			(hide yes)
@@
 			)
 		)
-		(property "Footprint" "sw_led:SW_MX_1u_SK6812MINI-E_ROTATE"
+		(property "Footprint" "sw_led:SW_MX_1u_SK6812MINI-E"
 			(at 320.04 287.02 0)
 			(hide yes)
@@
 			)
 		)
-		(property "Footprint" "sw_led:SW_MX_1u_SK6812MINI-E_ROTATE"
+		(property "Footprint" "sw_led:SW_MX_1u_SK6812MINI-E"
 			(at 198.12 203.2 0)
 			(hide yes)
@@
 			)
 		)
-		(property "Footprint" "sw_led:SW_MX_1u_SK6812MINI-E_ROTATE"
+		(property "Footprint" "sw_led:SW_MX_1u_SK6812MINI-E"
 			(at 167.64 370.84 0)
 			(hide yes)
@@
 			)
 		)
-		(property "Footprint" "sw_led:SW_MX_1u_SK6812MINI-E_ROTATE"
+		(property "Footprint" "sw_led:SW_MX_1u_SK6812MINI-E"
 			(at 320.04 119.38 0)
 			(hide yes)
@@
 			)
 		)
-		(property "Footprint" "sw_led:SW_MX_1u_SK6812MINI-E_ROTATE"
+		(property "Footprint" "sw_led:SW_MX_1u_SK6812MINI-E"
 			(at 137.16 287.02 0)
 			(hide yes)
@@
 			)
 		)
-		(property "Footprint" "sw_led:SW_MX_1u_SK6812MINI-E_ROTATE"
+		(property "Footprint" "sw_led:SW_MX_1u_SK6812MINI-E"
 			(at 320.04 203.2 0)
 			(hide yes)
@@
 			)
 		)
-		(property "Footprint" "sw_led:SW_MX_1u_SK6812MINI-E_ROTATE"
+		(property "Footprint" "sw_led:SW_MX_1u_SK6812MINI-E"
 			(at 228.6 203.2 0)
 			(hide yes)
@@
 			)
 		)
-		(property "Footprint" "sw_led:SW_MX_1u_SK6812MINI-E_ROTATE"
+		(property "Footprint" "sw_led:SW_MX_1u_SK6812MINI-E"
 			(at 259.08 287.02 0)
 			(hide yes)
@@
 			)
 		)
-		(property "Footprint" "sw_led:SW_MX_1u_SK6812MINI-E_ROTATE"
+		(property "Footprint" "sw_led:SW_MX_1u_SK6812MINI-E"
 			(at 76.2 35.56 0)
 			(hide yes)
@@
 			)
 		)
-		(property "Footprint" "sw_led:SW_MX_1u_SK6812MINI-E_ROTATE"
+		(property "Footprint" "sw_led:SW_MX_1u_SK6812MINI-E"
 			(at 106.68 287.02 0)
 			(hide yes)
@@
 			)
 		)
-		(property "Footprint" "sw_led:SW_MX_1u_SK6812MINI-E_ROTATE"
+		(property "Footprint" "sw_led:SW_MX_1u_SK6812MINI-E"
 			(at 198.12 370.84 0)
 			(hide yes)
@@
 			)
 		)
-		(property "Footprint" "sw_led:SW_MX_1u_SK6812MINI-E_ROTATE"
+		(property "Footprint" "sw_led:SW_MX_1u_SK6812MINI-E"
 			(at 289.56 370.84 0)
 			(hide yes)
@@
 			)
 		)
-		(property "Footprint" "sw_led:SW_MX_1u_SK6812MINI-E_ROTATE"
+		(property "Footprint" "sw_led:SW_MX_1u_SK6812MINI-E"
 			(at 76.2 119.38 0)
 			(hide yes)
@@
 			)
 		)
-		(property "Footprint" "sw_led:SW_MX_1u_SK6812MINI-E_ROTATE"
+		(property "Footprint" "sw_led:SW_MX_1u_SK6812MINI-E"
 			(at 137.16 370.84 0)
 			(hide yes)
@@
 			)
 		)
-		(property "Footprint" "sw_led:SW_MX_1u_SK6812MINI-E_ROTATE"
+		(property "Footprint" "sw_led:SW_MX_1u_SK6812MINI-E"
 			(at 137.16 35.56 0)
 			(hide yes)
@@
 			)
 		)
-		(property "Footprint" "sw_led:SW_MX_1u_SK6812MINI-E_ROTATE"
+		(property "Footprint" "sw_led:SW_MX_1u_SK6812MINI-E"
 			(at 76.2 370.84 0)
 			(hide yes)
@@
 			)
 		)
-		(property "Footprint" "sw_led:SW_MX_1u_SK6812MINI-E_ROTATE"
+		(property "Footprint" "sw_led:SW_MX_1u_SK6812MINI-E"
 			(at 45.72 370.84 0)
 			(hide yes)
@@
 			)
 		)
-		(property "Footprint" "sw_led:SW_MX_1u_SK6812MINI-E_ROTATE"
+		(property "Footprint" "sw_led:SW_MX_1u_SK6812MINI-E"
 			(at 106.68 203.2 0)
 			(hide yes)
@@
 			)
 		)
-		(property "Footprint" "sw_led:SW_MX_1u_SK6812MINI-E_ROTATE"
+		(property "Footprint" "sw_led:SW_MX_1u_SK6812MINI-E"
 			(at 167.64 287.02 0)
 			(hide yes)
@@
 			)
 		)
-		(property "Footprint" "sw_led:SW_MX_1u_SK6812MINI-E_ROTATE"
+		(property "Footprint" "sw_led:SW_MX_1u_SK6812MINI-E"
 			(at 198.12 287.02 0)
 			(hide yes)
