File: schema_2/schema_2.kicad_pcb (KiCad board)
At the start: 2 copper layers, 3.6 x 3.3 mm, 380 parts, among them J1 USB_C_Receptacle_PowerOnly_6P, J2 Conn_01x03_Pin, J3 Conn_01x04_Pin, SW103 SW_Push, SW104 SW_Push, SW105 SW_Push, SW21 SK12D07VG3, SW92 SK12D07VG3, U1 AP2112K-3.3, U2 W25Q128JVS, U3 74AHCT125, U4 STM32G070RBTx, U5 MAX98357A, U6 WEMOS_D1_mini, Y1 SX3M8.000M20F30TNN

Commit message: 30.10.2026 (1)
Parts:
- C1, C10, C100, C101, C102, C103, C104, C105, C106, C107, C108, C109, C11, C110, C111, C112, C113, C114, C115, C12, C13, C14, C15, C16, C17, C18, C19, C2, C20, C21, C22, C23, C24, C25, C26, C27, C28, C29, C3, C30, C31, C32, C33, C34, C35, C36, C37, C38, C39, C4, C40, C41, C42, C43, C44, C45, C46, C47, C48, C49, C5, C50, C51, C52, C53, C54, C55, C56, C57, C58, C59, C6, C60, C61, C62, C63, C64, C65, C66, C67, C68, C69, C7, C70, C71, C72, C73, C74, C75, C76, C77, C78, C79, C8, C80, C81, C82, C83, C84, C85, C86, C87, C88, C89, C9, C90, C91, C92, C93, C94, C95, C96, C97, C98, C99, D1, D10, D100, D101, D11, D12, D13, D14, D15, D16, D17, D18, D19, D2, D20, D21, D22, D23, D24, D25, D26, D27, D28, D29, D3, D30, D31, D32, D33, D34, D35, D36, D37, D38, D39, D4, D40, D41, D42, D43, D44, D45, D46, D47, D48, D49, D5, D50, D51, D52, D53, D54, D55, D56, D57, D58, D59, D6, D60, D61, D62, D63, D64, D65, D66, D67, D68, D69, D7, D70, D71, D72, D73, D74, D75, D76, D77, D78, D79, D8, D80, D81, D82, D83, D84, D85, D86, D87, D88, D89, D9, D90, D91, D92, D93, D94, D95, D96, D97, D98, D99, R1, R10, R11, R12, R13, R14, R15, R16, R17, R18, R19, R2, R20, R21, R22, R23, R24, R25, R26, R27, R28, R29, R3, R30, R31, R32, R33, R34, R35, R36, R37, R38, R39, R4, R40, R41, R42, R43, R44, R5, R6, R7, R8, R9, U1, U2, U3: moved to B.Cu
- LCD1: value ST7789_LCD -> ST7789_1.3_240x240_LCD_Module
- moved J3 329.9 mm to (374.4, -114.3)
- moved C1 304.5 mm to (541.3, -6.34), turned to 180 degrees
- moved C10 304.5 mm to (541.3, 20.7), turned to 180 degrees
- moved C11 304.5 mm to (541.3, 23.8), turned to 180 degrees
- moved C12 304.5 mm to (541.3, 26.8), turned to 180 degrees
- moved C13 304.5 mm to (541.3, 29.8), turned to 180 degrees
- moved C2 304.5 mm to (541.3, -3.33), turned to 180 degrees
- moved C4 304.5 mm to (541.3, 2.69), turned to 180 degrees
- moved C5 304.5 mm to (541.3, 5.70), turned to 180 degrees
- moved C7 304.5 mm to (541.3, 11.7), turned to 180 degrees
- moved C8 304.5 mm to (541.3, 14.7), turned to 180 degrees
- moved C3 304.5 mm to (541.3, -0.32), turned to 180 degrees
- moved C6 304.5 mm to (541.3, 8.71), turned to 180 degrees
- moved C9 304.5 mm to (541.3, 17.7), turned to 180 degrees
- moved D1 304.0 mm to (417.9, -54.2), turned to 180 degrees
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Connections:
- D10 pad 1: /col_5 -> /col_10
- D5 pad 1: /col_6 -> /col_5
- D6 pad 1: /col_7 -> /col_6
- D7 pad 1: /col_8 -> /col_7
- D8 pad 1: /col_9 -> /col_8
- D9 pad 1: /col_10 -> /col_9
- SW10 pad 6: Net-(D9-A) -> Net-(D10-A)
- SW5 pad 6: Net-(D10-A) -> Net-(D5-A)
- SW6 pad 6: Net-(D5-A) -> Net-(D6-A)
- SW7 pad 6: Net-(D6-A) -> Net-(D7-A)
- SW8 pad 6: Net-(D7-A) -> Net-(D8-A)
- SW9 pad 6: Net-(D8-A) -> Net-(D9-A)
Other:
- board size 3.6 x 3.3 mm -> 241 x 211 mm

Commit message: 30.10.2026 (2)
Parts:
- moved D1 373.3 mm to (55.5, 35.5)
- moved D2 353.1 mm to (75.5, 35.5)
- moved U4 304.1 mm to (263.5, 150.0)
- moved R11 242.5 mm to (312.1, 136.3)
- moved R12 242.5 mm to (312.1, 139.2)
- moved R14 242.5 mm to (312.1, 145.2)
- moved R16 242.5 mm to (312.1, 151.1)
- moved R17 242.5 mm to (312.1, 154.0)
- moved R2 242.5 mm to (316.6, 136.3)
- moved R20 242.5 mm to (307.7, 136.3)
- moved R21 242.5 mm to (307.7, 139.2)
- moved R23 242.5 mm to (307.7, 145.2)
- moved R25 242.5 mm to (307.7, 151.1)
- moved R26 242.5 mm to (307.7, 154.0)
- moved R29 242.5 mm to (303.3, 136.3)
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
Commit message: 30.10.2026 (3)
Parts:
- removed the LS1 at (426.6, -85.1)
- removed the U3 at (423.6, -113.7)
- removed the Y1 at (430.1, -85.1)
- R1: value R -> 1k
- SW21, SW92, U3, Y1: moved to B.Cu
- moved SW105 381.1 mm to (257.8, 169.1)
- moved SW92 368.1 mm to (276.9, 182.6), turned to -90 degrees
- moved SW103 353.9 mm to (251.5, 118.2)
- moved U5 353.5 mm to (272.7, 164.7), turned to -90 degrees
- moved SW104 338.8 mm to (267.8, 118.2)
- moved U2 327.1 mm to (250.4, 171.8), turned to 90 degrees
- moved LS1 310.3 mm to (276.1, 172.2), turned to -90 degrees
- moved J3 290.6 mm to (250.0, 148.3), turned to 180 degrees
- moved D82 289.6 mm to (55.5, 195.5)
- moved D11 287.6 mm to (55.5, 55.5)
- moved Y1 286.0 mm to (274.9, 152.4), turned to 180 degrees
- moved D92 283.4 mm to (55.5, 215.5)
- moved U3 282.6 mm to (249.0, 54.3)
- moved D93 282.5 mm to (75.5, 215.5)
- moved D72 281.4 mm to (55.5, 175.5)
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Connections:
- R13 pad 1: +5V -> +5VP
- R14 pad 1: +5V -> +5VP
- R15 pad 1: +5V -> +5VP

Commit message: 30.10.2026 (4)
Parts:
- moved C1 374.6 mm to (55.5, 54.5)
- moved R23 252.0 mm to (65.5, 75.5), turned to 0 degrees
- moved R22 232.0 mm to (85.5, 75.5), turned to 0 degrees
- moved R21 212.1 mm to (105.5, 75.5)
- moved R20 186.7 mm to (125.5, 95.5), turned to 0 degrees
- moved R19 166.6 mm to (145.5, 95.5), turned to 0 degrees
- moved C58 154.4 mm to (274.1, 143.3), turned to 0 degrees
- moved C59 152.2 mm to (274.1, 141.3), turned to 0 degrees
- moved R17 151.6 mm to (165.5, 115.5), turned to 0 degrees
- moved C115 137.6 mm to (274.8, 157.3), turned to 0 degrees
- moved R16 131.5 mm to (185.5, 115.5), turned to 0 degrees
- moved R30 97.9 mm to (205.5, 135.5), turned to 0 degrees
- moved R29 77.8 mm to (225.5, 135.5), turned to 0 degrees
- moved R24 64.7 mm to (244.0, 137.0), turned to -90 degrees
- moved R44 41.6 mm to (261.1, 171.3), turned to 90 degrees
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